Commit message: updated from old ws

File: catkin_ws/src/control/astra_description/urdf/astra.urdf.xacro (robot description, xacro)
@@ -318,5 +318,5 @@
 		<origin xyz="${link2_attach_point}" rpy="0 ${pi/2} 0" />
 		<axis xyz="0 1 0"/>
-		<limit effort="10" velocity="0.2" lower="-1.1" upper="1"/>
+		<limit effort="10" velocity="0.2" lower="-0.7" upper="0.6"/>
 	</joint>
 	<!-- joint4 -->
@@ -326,5 +326,5 @@
 		<origin xyz="${link3_attach_point}" />
 		<axis xyz="0 0 1"/>
-		<limit effort="10" velocity="0.2" lower="${(pi*-2)}" upper="${(pi*2)}"/>
+		<limit effort="10" velocity="0.2" lower="${(pi/-2)}" upper="${(pi/2)}"/>
 	</joint>
 	<!-- joint5 -->

Commit message: reference orientation+position

File: catkin_ws/src/control/astra_description/urdf/astra.urdf.xacro (robot description, xacro)
@@ -326,5 +326,5 @@
 		<origin xyz="${link3_attach_point}" />
 		<axis xyz="0 0 1"/>
-		<limit effort="10" velocity="0.2" lower="${(pi/-2)}" upper="${(pi/2)}"/>
+		<limit effort="10" velocity="0.2" lower="${(pi/-1)}" upper="${(pi/1)}"/>
 	</joint>
 	<!-- joint5 -->

Commit message: e

File: catkin_ws/src/control/astra_description/urdf/astra.urdf.xacro (robot description, xacro)
@@ -326,5 +326,5 @@
 		<origin xyz="${link3_attach_point}" />
 		<axis xyz="0 0 1"/>
-		<limit effort="10" velocity="0.2" lower="${(pi/-1)}" upper="${(pi/1)}"/>
+		<limit effort="10" velocity="0.2" lower="${(pi/-2)}" upper="${(pi/2)}"/>
 	</joint>
 	<!-- joint5 -->
@@ -342,5 +342,5 @@
 		<origin xyz="${link5_attach_point}" />
 		<axis xyz="0 0 1"/>
-		<limit effort="10" velocity="0.2" lower="${-(pi)}" upper="${pi}"/>
+		<limit effort="10" velocity="0.2" lower="${-(pi)}" upper="${pi/2}"/>
 	</joint>
 	<!-- gripper_left_finger_joint -->

Commit message: kkk

File: catkin_ws/src/control/astra_description/urdf/astra.urdf.xacro (robot description, xacro)
@@ -294,5 +294,5 @@
 		<origin xyz="${base_link_attach_point}" />
 		<axis xyz="0 0 1"/>
-		<limit effort="10" velocity="0.2" lower="${(pi*-2)}" upper="${(pi*2)}"/>
+		<limit effort="10" velocity="0.2" lower="${(pi*-3/4)}" upper="${(pi*3/4)}"/>
 	</joint>
 	<!-- joint2 -->
@@ -318,5 +318,5 @@
 		<origin xyz="${link2_attach_point}" rpy="0 ${pi/2} 0" />
 		<axis xyz="0 1 0"/>
-		<limit effort="10" velocity="0.2" lower="-0.7" upper="0.6"/>
+		<limit effort="10" velocity="0.2" lower="-1.1" upper="1.3"/>
 	</joint>
 	<!-- joint4 -->
@@ -334,5 +334,5 @@
 		<origin xyz="${link4_attach_point}" />
 		<axis xyz="0 1 0"/>
-		<limit effort="10" velocity="0.2" lower="-1.9" upper="1.9"/>
+		<limit effort="10" velocity="0.2" lower="-2.3" upper="2.8"/>
 	</joint>
 	<!-- joint6 -->
@@ -342,5 +342,5 @@
 		<origin xyz="${link5_attach_point}" />
 		<axis xyz="0 0 1"/>
-		<limit effort="10" velocity="0.2" lower="${-(pi)}" upper="${pi/2}"/>
+		<limit effort="10" velocity="0.2" lower="${-4.2}" upper="${3.8}"/>
 	</joint>
 	<!-- gripper_left_finger_joint -->

Commit message: begin inverse

File: catkin_ws/src/control/astra_description/urdf/astra.urdf.xacro (robot description, xacro)
@@ -334,5 +334,5 @@
 		<origin xyz="${link4_attach_point}" />
 		<axis xyz="0 1 0"/>
-		<limit effort="10" velocity="0.2" lower="-2.3" upper="2.8"/>
+		<limit effort="10" velocity="0.2" lower="-2.8" upper="2.3"/>
 	</joint>
 	<!-- joint6 -->
