Commit message: manual merge of changes from humble branch

File: hd_ws/src/control/kerby_moveit_config/config/kerby.ros2_control.xacro (robot description, xacro)
@@ -7,9 +7,7 @@
                 <!-- By default, set up controllers for simulation. This won't work on real hardware -->
                 <plugin>kerby_hw_interface/KerbyArmInterface</plugin>
-                <!--  gazebo_ros2_control/GazeboSystem    mock_components/GenericSystem   kerby_hw_interface/KerbyArmInterface  -->
             </hardware>
             <joint name="joint1">
                 <command_interface name="position"/>
-                <!-- <command_interface name="velocity"/> -->
                 <state_interface name="position">
                   <param name="initial_value">${initial_positions['joint1']}</param>
@@ -19,5 +17,4 @@
             <joint name="joint2">
                 <command_interface name="position"/>
-                <!-- <command_interface name="velocity"/> -->
                 <state_interface name="position">
                   <param name="initial_value">${initial_positions['joint2']}</param>
@@ -27,5 +24,4 @@
             <joint name="joint3">
                 <command_interface name="position"/>
-                <!-- <command_interface name="velocity"/> -->
                 <state_interface name="position">
                   <param name="initial_value">${initial_positions['joint3']}</param>
@@ -35,5 +31,4 @@
             <joint name="joint4">
                 <command_interface name="position"/>
-                <!-- <command_interface name="velocity"/> -->
                 <state_interface name="position">
                   <param name="initial_value">${initial_positions['joint4']}</param>
@@ -43,5 +38,4 @@
             <joint name="joint5">
                 <command_interface name="position"/>
-                <!-- <command_interface name="velocity"/> -->
                 <state_interface name="position">
                   <param name="initial_value">${initial_positions['joint5']}</param>
@@ -51,5 +45,4 @@
             <joint name="joint6">
                 <command_interface name="position"/>
-                <!-- <command_interface name="velocity"/> -->
                 <state_interface name="position">
                   <param name="initial_value">${initial_positions['joint6']}</param>
@@ -57,18 +50,5 @@
                 <state_interface name="velocity"/>
             </joint>
-            <joint name="gripper_left_finger_joint">
-                <command_interface name="position"/>
-                <!-- <command_interface name="velocity"/> -->
-                <state_interface name="position">
-                  <param name="initial_value">${initial_positions['gripper_left_finger_joint']}</param>
-                </state_interface>
-                <state_interface name="velocity"/>
-            </joint>
         </ros2_control>
-    <gazebo>
-      <plugin name="gazebo_ros2_control" filename="libgazebo_ros2_control.so">
-        <parameters>$(find kerby_moveit_config)/config/ros2_controllers.yaml</parameters>
-      </plugin>
-    </gazebo>
     </xacro:macro>
 </robot>

Commit message: added second set of controllers + hardware interface to keep track of the rest of the rover state

File: hd_ws/src/control/kerby_moveit_config/config/kerby.ros2_control.xacro (robot description, xacro)
@@ -1,9 +1,8 @@
 <?xml version="1.0"?>
 <robot xmlns:xacro="http://www.ros.org/wiki/xacro">
-    <xacro:macro name="kerby_ros2_control" params="name initial_positions_file">
+    <xacro:macro name="kerby_arm_ros2_control" params="name initial_positions_file">
         <xacro:property name="initial_positions" value="${load_yaml(initial_positions_file)['initial_positions']}"/>
         <ros2_control name="${name}" type="system">
             <hardware>
-                <!-- By default, set up controllers for simulation. This won't work on real hardware -->
                 <plugin>kerby_hw_interface/KerbyArmInterface</plugin>
             </hardware>
@@ -59,3 +58,71 @@
         </ros2_control>
     </xacro:macro>
+    <xacro:macro name="kerby_left_ros2_control" params="name initial_positions_file">
+        <xacro:property name="initial_positions" value="${load_yaml(initial_positions_file)['initial_positions']}"/>
+        <ros2_control name="${name}" type="system">
+            <hardware>
+                <plugin>kerby_hw_interface/KerbyBaseInterface</plugin>
+            </hardware>
+            <joint name="pivot_gauche">
+                <command_interface name="position"/>
+                <state_interface name="position">
+                  <param name="initial_value">${initial_positions['pivot_gauche']}</param>
+                </state_interface>
+            </joint>
+            <joint name="steering1">
+                <command_interface name="position"/>
+                <state_interface name="position">
+                  <param name="initial_value">${initial_positions['steering1']}</param>
+                </state_interface>
+            </joint>
+            <joint name="driving1">
+                <command_interface name="position"/>
+                <state_interface name="position">
+                  <param name="initial_value">${initial_positions['driving1']}</param>
+                </state_interface>
+            </joint>
+            <joint name="steering4">
+                <command_interface name="position"/>
+                <state_interface name="position">
+                  <param name="initial_value">${initial_positions['driving1']}</param>
+                </state_interface>
+            </joint>
+            <joint name="driving4">
+                <command_interface name="position"/>
+                <state_interface name="position">
+                  <param name="initial_value">${initial_positions['driving1']}</param>
+                </state_interface>
+            </joint>
+            <joint name="pivot_droit">
+                <command_interface name="position"/>
+                <state_interface name="position">
+                  <param name="initial_value">${initial_positions['driving1']}</param>
+                </state_interface>
+            </joint>
+            <joint name="steering2">
+                <command_interface name="position"/>
+                <state_interface name="position">
+                  <param name="initial_value">${initial_positions['driving1']}</param>
+                </state_interface>
+            </joint>
+            <joint name="driving2">
+                <command_interface name="position"/>
+                <state_interface name="position">
+                  <param name="initial_value">${initial_positions['driving1']}</param>
+                </state_interface>
+            </joint>
+            <joint name="steering3">
+                <command_interface name="position"/>
+                <state_interface name="position">
+                  <param name="initial_value">${initial_positions['driving1']}</param>
+                </state_interface>
+            </joint>
+            <joint name="driving3">
+                <command_interface name="position"/>
+                <state_interface name="position">
+                  <param name="initial_value">${initial_positions['driving1']}</param>
+                </state_interface>
+            </joint>
+        </ros2_control>
+    </xacro:macro>
 </robot>

File: hd_ws/src/control/kerby_moveit_config/config/kerby.urdf.xacro (robot description, xacro)
@@ -6,4 +6,5 @@
     <!-- Import control_xacro -->
     <xacro:include filename="kerby.ros2_control.xacro" />
-    <xacro:kerby_ros2_control name="FakeSystem" initial_positions_file="$(arg initial_positions_file)"/>
+    <xacro:kerby_arm_ros2_control name="FakeSystem" initial_positions_file="$(arg initial_positions_file)"/>
+    <xacro:kerby_left_ros2_control name="FakeSystem" initial_positions_file="$(arg initial_positions_file)"/>
 </robot>

Commit message: cleanup

File: hd_ws/src/control/kerby_moveit_config/config/kerby.ros2_control.xacro (robot description, xacro)
@@ -58,5 +58,5 @@
         </ros2_control>
     </xacro:macro>
-    <xacro:macro name="kerby_left_ros2_control" params="name initial_positions_file">
+    <xacro:macro name="kerby_base_ros2_control" params="name initial_positions_file">
         <xacro:property name="initial_positions" value="${load_yaml(initial_positions_file)['initial_positions']}"/>
         <ros2_control name="${name}" type="system">
@@ -85,5 +85,5 @@
                 <command_interface name="position"/>
                 <state_interface name="position">
-                  <param name="initial_value">${initial_positions['driving1']}</param>
+                  <param name="initial_value">${initial_positions['steering4']}</param>
                 </state_interface>
             </joint>
@@ -91,5 +91,5 @@
                 <command_interface name="position"/>
                 <state_interface name="position">
-                  <param name="initial_value">${initial_positions['driving1']}</param>
+                  <param name="initial_value">${initial_positions['driving4']}</param>
                 </state_interface>
             </joint>
@@ -97,5 +97,5 @@
                 <command_interface name="position"/>
                 <state_interface name="position">
-                  <param name="initial_value">${initial_positions['driving1']}</param>
+                  <param name="initial_value">${initial_positions['pivot_droit']}</param>
                 </state_interface>
             </joint>
@@ -103,5 +103,5 @@
                 <command_interface name="position"/>
                 <state_interface name="position">
-                  <param name="initial_value">${initial_positions['driving1']}</param>
+                  <param name="initial_value">${initial_positions['steering2']}</param>
                 </state_interface>
             </joint>
@@ -109,5 +109,5 @@
                 <command_interface name="position"/>
                 <state_interface name="position">
-                  <param name="initial_value">${initial_positions['driving1']}</param>
+                  <param name="initial_value">${initial_positions['driving2']}</param>
                 </state_interface>
             </joint>
@@ -115,5 +115,5 @@
                 <command_interface name="position"/>
                 <state_interface name="position">
-                  <param name="initial_value">${initial_positions['driving1']}</param>
+                  <param name="initial_value">${initial_positions['steering3']}</param>
                 </state_interface>
             </joint>
@@ -121,5 +121,5 @@
                 <command_interface name="position"/>
                 <state_interface name="position">
-                  <param name="initial_value">${initial_positions['driving1']}</param>
+                  <param name="initial_value">${initial_positions['driving3']}</param>
                 </state_interface>
             </joint>

File: hd_ws/src/control/kerby_moveit_config/config/kerby.urdf.xacro (robot description, xacro)
@@ -7,4 +7,4 @@
     <xacro:include filename="kerby.ros2_control.xacro" />
     <xacro:kerby_arm_ros2_control name="FakeSystem" initial_positions_file="$(arg initial_positions_file)"/>
-    <xacro:kerby_left_ros2_control name="FakeSystem" initial_positions_file="$(arg initial_positions_file)"/>
+    <xacro:kerby_base_ros2_control name="FakeSystem" initial_positions_file="$(arg initial_positions_file)"/>
 </robot>
