Commit message: manual merge with foxy branch

File: hd_ws/src/control/kerby_description/urdf/materials.xacro (robot description, xacro)
@@ -11,8 +11,9 @@
 </material>
 <material name="pink">
-  <color rgba="1 0.4117 0.70588 1.000"/>
+  <!-- <color rgba="1 0.4117 0.70588 1.000"/> -->
+  <color rgba="1 1 1 1.000"/>
 </material>
 <material name="blue">
-  <color rgba="0 0 0.7 1.000"/>
+  <color rgba="0 0 0.5 1.000"/>
 </material>
 </robot>

File: hd_ws/src/control/kerby_moveit_config/config/kerby.ros2_control.xacro (robot description, xacro)
@@ -1,9 +1,8 @@
 <?xml version="1.0"?>
 <robot xmlns:xacro="http://www.ros.org/wiki/xacro">
-    <xacro:macro name="kerby_ros2_control" params="name initial_positions_file">
+    <xacro:macro name="kerby_arm_ros2_control" params="name initial_positions_file">
         <xacro:property name="initial_positions" value="${load_yaml(initial_positions_file)['initial_positions']}"/>
         <ros2_control name="${name}" type="system">
             <hardware>
-                <!-- By default, set up controllers for simulation. This won't work on real hardware -->
                 <plugin>kerby_hw_interface/KerbyArmInterface</plugin>
             </hardware>
@@ -50,4 +49,79 @@
                 <state_interface name="velocity"/>
             </joint>
+            <joint name="finger1">
+                <command_interface name="position"/>
+                <state_interface name="position">
+                  <param name="initial_value">${initial_positions['finger1']}</param>
+                </state_interface>
+                <state_interface name="velocity"/>
+            </joint>
+        </ros2_control>
+    </xacro:macro>
+    <xacro:macro name="kerby_base_ros2_control" params="name initial_positions_file">
+        <xacro:property name="initial_positions" value="${load_yaml(initial_positions_file)['initial_positions']}"/>
+        <ros2_control name="${name}" type="system">
+            <hardware>
+                <plugin>kerby_hw_interface/KerbyBaseInterface</plugin>
+            </hardware>
+            <joint name="pivot_gauche">
+                <command_interface name="position"/>
+                <state_interface name="position">
+                  <param name="initial_value">${initial_positions['pivot_gauche']}</param>
+                </state_interface>
+            </joint>
+            <joint name="steering1">
+                <command_interface name="position"/>
+                <state_interface name="position">
+                  <param name="initial_value">${initial_positions['steering1']}</param>
+                </state_interface>
+            </joint>
+            <joint name="driving1">
+                <command_interface name="position"/>
+                <state_interface name="position">
+                  <param name="initial_value">${initial_positions['driving1']}</param>
+                </state_interface>
+            </joint>
+            <joint name="steering4">
+                <command_interface name="position"/>
+                <state_interface name="position">
+                  <param name="initial_value">${initial_positions['steering4']}</param>
+                </state_interface>
+            </joint>
+            <joint name="driving4">
+                <command_interface name="position"/>
+                <state_interface name="position">
+                  <param name="initial_value">${initial_positions['driving4']}</param>
+                </state_interface>
+            </joint>
+            <joint name="pivot_droit">
+                <command_interface name="position"/>
+                <state_interface name="position">
+                  <param name="initial_value">${initial_positions['pivot_droit']}</param>
+                </state_interface>
+            </joint>
+            <joint name="steering2">
+                <command_interface name="position"/>
+                <state_interface name="position">
+                  <param name="initial_value">${initial_positions['steering2']}</param>
+                </state_interface>
+            </joint>
+            <joint name="driving2">
+                <command_interface name="position"/>
+                <state_interface name="position">
+                  <param name="initial_value">${initial_positions['driving2']}</param>
+                </state_interface>
+            </joint>
+            <joint name="steering3">
+                <command_interface name="position"/>
+                <state_interface name="position">
+                  <param name="initial_value">${initial_positions['steering3']}</param>
+                </state_interface>
+            </joint>
+            <joint name="driving3">
+                <command_interface name="position"/>
+                <state_interface name="position">
+                  <param name="initial_value">${initial_positions['driving3']}</param>
+                </state_interface>
+            </joint>
         </ros2_control>
     </xacro:macro>

File: hd_ws/src/control/kerby_moveit_config/config/kerby.urdf.xacro (robot description, xacro)
@@ -6,4 +6,5 @@
     <!-- Import control_xacro -->
     <xacro:include filename="kerby.ros2_control.xacro" />
-    <xacro:kerby_ros2_control name="FakeSystem" initial_positions_file="$(arg initial_positions_file)"/>
+    <xacro:kerby_arm_ros2_control name="FakeSystem" initial_positions_file="$(arg initial_positions_file)"/>
+    <xacro:kerby_base_ros2_control name="KerbyBaseSystem" initial_positions_file="$(arg initial_positions_file)"/>
 </robot>
