Commit message: renaming rrrr

File: hd_ws/src/control/kerby_description/urdf/kerby.urdf.xacro (robot description, xacro)
@@ -1,363 +1,521 @@
-<?xml version="1.0"?>
-<robot xmlns:xacro="http://www.ros.org/wiki/xacro" name="kerby">
-<!-- ======================================================================================================================== -->
-	<!-- ==========CONSANTS========== -->
-	<!-- base_link is rover -->
-	<!-- base_link constants -->
-	<xacro:property name="base_link_dim_x" value="0.6" />
-	<xacro:property name="base_link_dim_y" value="0.5" />
-	<xacro:property name="base_link_dim_z" value="0.16125" />
-	<xacro:property name="base_link_dim" value="0.6 0.5 0.16125" />
-	<xacro:property name="base_link_btm_shift_x" value="0" />
-	<xacro:property name="base_link_btm_shift_y" value="0" />
-	<xacro:property name="base_link_btm_shift_z" value="0" />
-	<xacro:property name="base_link_top_shift_x" value="${(0.525-(base_link_dim_x/2))}" />
-	<xacro:property name="base_link_top_shift_y" value="0" />
-	<xacro:property name="base_link_top_shift_z" value="${(base_link_dim_z/2)}" />
-	<xacro:property name="base_link_origin" value="0 0 0" />
-	<xacro:property name="base_link_attach_point" value="${((0.525-(base_link_dim_x/2))+0)} 0 ${((base_link_dim_z/2)+0)}" />
-	<!-- link1 constants -->
-	<xacro:property name="link1_dim_x" value="0.08" />
-	<xacro:property name="link1_dim_y" value="0.1505" />
-	<xacro:property name="link1_dim_z" value="0.138" />
-	<xacro:property name="link1_dim" value="0.08 0.1505 0.138" />
-	<xacro:property name="link1_btm_shift_x" value="0" />
-	<xacro:property name="link1_btm_shift_y" value="${-((0.094-(link1_dim_y/2)))}" />
-	<xacro:property name="link1_btm_shift_z" value="${(link1_dim_z/2)}" />
-	<xacro:property name="link1_top_shift_x" value="0" />
-	<xacro:property name="link1_top_shift_y" value="${(link1_dim_x-0.0565)}" />
-	<xacro:property name="link1_top_shift_z" value="${(0.098-(link1_dim_z/2))}" />
-	<xacro:property name="link1_origin" value="0 ${-((0.094-(link1_dim_y/2)))} ${(link1_dim_z/2)}" />
-	<xacro:property name="link1_attach_point" value="0 ${((link1_dim_x-0.0565)+-((0.094-(link1_dim_y/2))))} ${((0.098-(link1_dim_z/2))+(link1_dim_z/2))}" />
-	<!-- link2 constants -->
-	<xacro:property name="link2_dim_x" value="0.096" />
-	<xacro:property name="link2_dim_y" value="0.07" />
-	<xacro:property name="link2_dim_z" value="0.487225" />
-	<xacro:property name="link2_dim" value="0.096 0.07 0.487225" />
-	<xacro:property name="link2_btm_shift_x" value="0" />
-	<xacro:property name="link2_btm_shift_y" value="0" />
-	<xacro:property name="link2_btm_shift_z" value="${-((0.048-(link2_dim_z/2)))}" />
-	<xacro:property name="link2_top_shift_x" value="${(0.039225-(link2_dim_x/2))}" />
-	<xacro:property name="link2_top_shift_y" value="0" />
-	<xacro:property name="link2_top_shift_z" value="${((link2_dim_z/2)-0.039225)}" />
-	<xacro:property name="link2_origin" value="0 0 ${-((0.048-(link2_dim_z/2)))}" />
-	<xacro:property name="link2_attach_point" value="${((0.039225-(link2_dim_x/2))+0)} 0 ${(((link2_dim_z/2)-0.039225)+-((0.048-(link2_dim_z/2))))}" />
-	<!-- motor_j3 constants -->
-	<xacro:property name="motor_j3_dim_x" value="0.09" />
-	<xacro:property name="motor_j3_dim_y" value="0.07" />
-	<xacro:property name="motor_j3_dim_z" value="0.3" />
-	<xacro:property name="motor_j3_dim" value="0.09 0.07 0.3" />
-	<xacro:property name="motor_j3_btm_shift_x" value="-0.084225" />
-	<xacro:property name="motor_j3_btm_shift_y" value="0" />
-	<xacro:property name="motor_j3_btm_shift_z" value="0.004388" />
-	<xacro:property name="motor_j3_top_shift_x" value="0" />
-	<xacro:property name="motor_j3_top_shift_y" value="0" />
-	<xacro:property name="motor_j3_top_shift_z" value="0" />
-	<xacro:property name="motor_j3_origin" value="-0.084225 0 0.004388" />
-	<xacro:property name="motor_j3_attach_point" value="-0.084225 0 0.004388" />
-	<!-- link3 constants -->
-	<xacro:property name="link3_dim_x" value="0.115" />
-	<xacro:property name="link3_dim_y" value="0.112" />
-	<xacro:property name="link3_dim_z" value="0.387" />
-	<xacro:property name="link3_dim" value="0.115 0.112 0.387" />
-	<xacro:property name="link3_btm_shift_x" value="${(0.02-(link3_dim_x/2))}" />
-	<xacro:property name="link3_btm_shift_y" value="0" />
-	<xacro:property name="link3_btm_shift_z" value="${-((0.087-(link3_dim_z/2)))}" />
-	<xacro:property name="link3_top_shift_x" value="${(0.0415-(link3_dim_x/2))}" />
-	<xacro:property name="link3_top_shift_y" value="0" />
-	<xacro:property name="link3_top_shift_z" value="${(link3_dim_z/2)}" />
-	<xacro:property name="link3_origin" value="${(0.02-(link3_dim_x/2))} 0 ${-((0.087-(link3_dim_z/2)))}" />
-	<xacro:property name="link3_attach_point" value="${((0.0415-(link3_dim_x/2))+(0.02-(link3_dim_x/2)))} 0 ${((link3_dim_z/2)+-((0.087-(link3_dim_z/2))))}" />
-	<!-- link4 constants -->
-	<xacro:property name="link4_dim_x" value="0.08" />
-	<xacro:property name="link4_dim_y" value="0.175" />
-	<xacro:property name="link4_dim_z" value="0.1208" />
-	<xacro:property name="link4_dim" value="0.08 0.175 0.1208" />
-	<xacro:property name="link4_btm_shift_x" value="0" />
-	<xacro:property name="link4_btm_shift_y" value="0" />
-	<xacro:property name="link4_btm_shift_z" value="${(link4_dim_z/2)}" />
-	<xacro:property name="link4_top_shift_x" value="0" />
-	<xacro:property name="link4_top_shift_y" value="0" />
-	<xacro:property name="link4_top_shift_z" value="${((link4_dim_z/2)-0.031)}" />
-	<xacro:property name="link4_origin" value="0 0 ${(link4_dim_z/2)}" />
-	<xacro:property name="link4_attach_point" value="0 0 ${(((link4_dim_z/2)-0.031)+(link4_dim_z/2))}" />
-	<!-- link5 constants -->
-	<xacro:property name="link5_dim_x" value="0.045" />
-	<xacro:property name="link5_dim_y" value="0.045" />
-	<xacro:property name="link5_dim_z" value="0.09455" />
-	<xacro:property name="link5_dim" value="0.045 0.045 0.09455" />
-	<xacro:property name="link5_btm_shift_x" value="0" />
-	<xacro:property name="link5_btm_shift_y" value="0" />
-	<xacro:property name="link5_btm_shift_z" value="${((link5_dim_z/2)-0.0318)}" />
-	<xacro:property name="link5_top_shift_x" value="0" />
-	<xacro:property name="link5_top_shift_y" value="0" />
-	<xacro:property name="link5_top_shift_z" value="${(link5_dim_z/2)}" />
-	<xacro:property name="link5_origin" value="0 0 ${((link5_dim_z/2)-0.0318)}" />
-	<xacro:property name="link5_attach_point" value="0 0 ${    0.103+0.045+    ((link5_dim_z/2)+((link5_dim_z/2)-0.0318))}" />
-	<!-- gripper_base constants -->
-	<xacro:property name="gripper_base_dim_x" value="0.1565" />
-	<xacro:property name="gripper_base_dim_y" value="0.125" />
-	<xacro:property name="gripper_base_dim_z" value="0.103" />
-	<xacro:property name="gripper_base_dim" value="0.1565 0.125 0.103" />
-	<xacro:property name="gripper_base_btm_shift_x" value="${((gripper_base_dim_x/2)-0.076)}" />
-	<xacro:property name="gripper_base_btm_shift_y" value="${-((0.0671-(gripper_base_dim_y/2)))}" />
-	<xacro:property name="gripper_base_btm_shift_z" value="${(gripper_base_dim_z/2)}" />
-	<xacro:property name="gripper_base_top_shift_x" value="${-(((gripper_base_dim_x/2)-0.076))}" />
-	<xacro:property name="gripper_base_top_shift_y" value="${(0.0671-(gripper_base_dim_y/2))}" />
-	<xacro:property name="gripper_base_top_shift_z" value="${(gripper_base_dim_z/2)}" />
-	<xacro:property name="gripper_base_origin" value="${((gripper_base_dim_x/2)-0.076)} ${-((0.0671-(gripper_base_dim_y/2)))} ${(    -0.045-    gripper_base_dim_z/2)}" />
-	<xacro:property name="gripper_base_attach_point" value="${(-(((gripper_base_dim_x/2)-0.076))+((gripper_base_dim_x/2)-0.076))} ${((0.0671-(gripper_base_dim_y/2))+-((0.0671-(gripper_base_dim_y/2))))} ${(    -0.045-    (gripper_base_dim_z/2)+(gripper_base_dim_z/2))}" />
-	<!-- gripper_left_finger constants -->
-	<xacro:property name="gripper_left_finger_dim_x" value="0.0215" />
-	<xacro:property name="gripper_left_finger_dim_y" value="0.016" />
-	<xacro:property name="gripper_left_finger_dim_z" value="0.045" />
-	<xacro:property name="gripper_left_finger_dim" value="0.0215 0.016 0.045" />
-	<xacro:property name="gripper_left_finger_btm_shift_x" value="0" />
-	<xacro:property name="gripper_left_finger_btm_shift_y" value="${(gripper_left_finger_dim_y/2)}" />
-	<xacro:property name="gripper_left_finger_btm_shift_z" value="${(gripper_left_finger_dim_z/2)}" />
-	<xacro:property name="gripper_left_finger_top_shift_x" value="0" />
-	<xacro:property name="gripper_left_finger_top_shift_y" value="0" />
-	<xacro:property name="gripper_left_finger_top_shift_z" value="0" />
-	<xacro:property name="gripper_left_finger_origin" value="0 ${(gripper_left_finger_dim_y/2)} ${(gripper_left_finger_dim_z/2)}" />
-	<xacro:property name="gripper_left_finger_attach_point" value="0 ${((gripper_left_finger_dim_y/2)+0)} ${((gripper_left_finger_dim_z/2)+0)}" />
-	<!-- gripper_right_finger constants -->
-	<xacro:property name="gripper_right_finger_dim_x" value="0.0215" />
-	<xacro:property name="gripper_right_finger_dim_y" value="0.016" />
-	<xacro:property name="gripper_right_finger_dim_z" value="0.045" />
-	<xacro:property name="gripper_right_finger_dim" value="0.0215 0.016 0.045" />
-	<xacro:property name="gripper_right_finger_btm_shift_x" value="0" />
-	<xacro:property name="gripper_right_finger_btm_shift_y" value="${(-(gripper_right_finger_dim_y)/2)}" />
-	<xacro:property name="gripper_right_finger_btm_shift_z" value="${(gripper_right_finger_dim_z/2)}" />
-	<xacro:property name="gripper_right_finger_top_shift_x" value="0" />
-	<xacro:property name="gripper_right_finger_top_shift_y" value="0" />
-	<xacro:property name="gripper_right_finger_top_shift_z" value="0" />
-	<xacro:property name="gripper_right_finger_origin" value="0 ${(-(gripper_right_finger_dim_y)/2)} ${(gripper_right_finger_dim_z/2)}" />
-	<xacro:property name="gripper_right_finger_attach_point" value="0 ${((-(gripper_right_finger_dim_y)/2)+0)} ${((gripper_right_finger_dim_z/2)+0)}" />
-	<!-- ======================================================================================================================== -->
-	<!-- ==========LINKS========== -->
-	<!-- base_link -->
-	<link name="base_link">
-		<visual>
-			<geometry>
-				<box size="${base_link_dim}"/>
-			</geometry>
-			<origin xyz="${base_link_origin}" />
-		</visual>
-		<collision>
-			<geometry>
-				<box size="${base_link_dim}"/>
-			</geometry>
-			<origin xyz="${base_link_origin}" />
-		</collision>
-	</link>
-	<!-- link1 -->
-	<link name="link1">
-		<visual>
-			<geometry>
-				<box size="${link1_dim}"/>
-			</geometry>
-			<origin xyz="${link1_origin}" />
-		</visual>
-		<collision>
-			<geometry>
-				<box size="${link1_dim}"/>
-			</geometry>
-			<origin xyz="${link1_origin}" />
-		</collision>
-	</link>
-	<!-- link2 -->
-	<link name="link2">
-		<visual>
-			<geometry>
-				<box size="${link2_dim}"/>
-			</geometry>
-			<origin xyz="${link2_origin}" />
-		</visual>
-		<collision>
-			<geometry>
-				<box size="${link2_dim}"/>
-			</geometry>
-			<origin xyz="${link2_origin}" />
-		</collision>
-	</link>
-	<!-- motor_j3 -->
-	<link name="motor_j3">
-		<visual>
-			<geometry>
-				<box size="${motor_j3_dim}"/>
-			</geometry>
-			<origin xyz="${motor_j3_origin}" />
-		</visual>
-		<collision>
-			<geometry>
-				<box size="${motor_j3_dim}"/>
-			</geometry>
-			<origin xyz="${motor_j3_origin}" />
-		</collision>
-	</link>
-	<!-- link3 -->
-	<link name="link3">
-		<visual>
-			<geometry>
-				<box size="${link3_dim}"/>
-			</geometry>
-			<origin xyz="${link3_origin}" />
-		</visual>
-		<collision>
-			<geometry>
-				<box size="${link3_dim}"/>
-			</geometry>
-			<origin xyz="${link3_origin}" />
-		</collision>
-	</link>
-	<!-- link4 -->
-	<link name="link4">
-		<visual>
-			<geometry>
-				<box size="${link4_dim}"/>
-			</geometry>
-			<origin xyz="${link4_origin}" />
-		</visual>
-		<collision>
-			<geometry>
-				<box size="${link4_dim}"/>
-			</geometry>
-			<origin xyz="${link4_origin}" />
-		</collision>
-	</link>
-	<!-- link5 -->
-	<link name="link5">
-		<visual>
-			<geometry>
-				<box size="${link5_dim}"/>
-			</geometry>
-			<origin xyz="${link5_origin}" />
-		</visual>
-		<collision>
-			<geometry>
-				<box size="${link5_dim}"/>
-			</geometry>
-			<origin xyz="${link5_origin}" />
-		</collision>
-	</link>
-	<!-- gripper_base -->
-	<link name="gripper_base">
-		<visual>
-			<geometry>
-				<box size="${gripper_base_dim}"/>
-			</geometry>
-			<origin xyz="${gripper_base_origin}" />
-		</visual>
-		<collision>
-			<geometry>
-				<box size="${gripper_base_dim}"/>
-			</geometry>
-			<origin xyz="${gripper_base_origin}" />
-		</collision>
-	</link>
-	<!-- gripper_left_finger -->
-	<link name="gripper_left_finger">
-		<visual>
-			<geometry>
-				<box size="${gripper_left_finger_dim}"/>
-			</geometry>
-			<origin xyz="${gripper_left_finger_origin}" />
-		</visual>
-		<collision>
-			<geometry>
-				<box size="${gripper_left_finger_dim}"/>
-			</geometry>
-			<origin xyz="${gripper_left_finger_origin}" />
-		</collision>
-	</link>
-	<!-- gripper_right_finger -->
-	<link name="gripper_right_finger">
-		<visual>
-			<geometry>
-				<box size="${gripper_right_finger_dim}"/>
-			</geometry>
-			<origin xyz="${gripper_right_finger_origin}" />
-		</visual>
-		<collision>
-			<geometry>
-				<box size="${gripper_right_finger_dim}"/>
-			</geometry>
-			<origin xyz="${gripper_right_finger_origin}" />
-		</collision>
-	</link>
-	<!-- ======================================================================================================================== -->
-	<!-- ==========JOINTS========== -->
-	<!-- joint1 -->
-	<joint name="joint1" type="revolute">
-		<parent link="base_link"/>
-		<child link="link1"/>
-		<origin xyz="${base_link_attach_point}" />
-		<axis xyz="0 0 1"/>
-		<limit effort="10" velocity="0.2" lower="${(pi*-3/4)}" upper="${(pi*3/4)}"/>
-	</joint>
-	<!-- joint2 -->
-	<joint name="joint2" type="revolute">
-		<parent link="link1"/>
-		<child link="link2"/>
-		<origin xyz="${link1_attach_point}" />
-		<axis xyz="0 1 0"/>
-		<limit effort="10" velocity="0.2" lower="-1.34" upper="2.07"/>
-	</joint>
-	<!-- motor_j3_joint -->
-	<joint name="motor_j3_joint" type="fixed">
-		<parent link="link2"/>
-		<child link="motor_j3"/>
-		<origin xyz="${link2_attach_point}" />
-		<axis xyz="1 0 0"/>
-		<limit effort="1" velocity="0.2" lower="${-(pi)}" upper="${pi}"/>
-	</joint>
-	<!-- joint3 -->
-	<joint name="joint3" type="revolute">
-		<parent link="link2"/>
-		<child link="link3"/>
-		<origin xyz="${link2_attach_point}" rpy="0 ${pi/2} 0" />
-		<axis xyz="0 1 0"/>
-		<limit effort="10" velocity="0.2" lower="-1.1" upper="1.3"/>
-	</joint>
-	<!-- joint4 -->
-	<joint name="joint4" type="revolute">
-		<parent link="link3"/>
-		<child link="link4"/>
-		<origin xyz="${link3_attach_point}" />
-		<axis xyz="0 0 1"/>
-		<limit effort="10" velocity="0.2" lower="${(pi/-2)}" upper="${(pi/2)}"/>
-	</joint>
-	<!-- joint5 -->
-	<joint name="joint5" type="revolute">
-		<parent link="link4"/>
-		<child link="link5"/>
-		<origin xyz="${link4_attach_point}" />
-		<axis xyz="0 1 0"/>
-		<limit effort="10" velocity="0.2" lower="-2.8" upper="2.3"/>
-	</joint>
-	<!-- joint6 -->
-	<joint name="joint6" type="revolute">
-		<parent link="link5"/>
-		<child link="gripper_base"/>
-		<origin xyz="${link5_attach_point}" />
-		<axis xyz="0 0 1"/>
-		<limit effort="10" velocity="0.2" lower="${-4.2}" upper="${3.8}"/>
-	</joint>
-	<!-- gripper_left_finger_joint -->
-	<joint name="gripper_left_finger_joint" type="prismatic">
-		<parent link="gripper_base"/>
-		<child link="gripper_left_finger"/>
-		<origin xyz="${gripper_base_attach_point}" />
-		<axis xyz="0 1 0"/>
-		<limit effort="1" velocity="0.5" lower="0" upper="0.04"/>
-	</joint>
-	<!-- gripper_right_finger_joint -->
-	<joint name="gripper_right_finger_joint" type="prismatic">
-		<parent link="gripper_base"/>
-		<child link="gripper_right_finger"/>
-		<origin xyz="${gripper_base_attach_point}" />
-		<axis xyz="0 1 0"/>
-		<limit effort="1" velocity="0.5" lower="0" upper="0.1"/>
-		<mimic joint="gripper_left_finger_joint" multiplier="-1" offset="0"/>
-	</joint>
+<?xml version="1.0" ?>
+<robot name="kerby" xmlns:xacro="http://www.ros.org/wiki/xacro">
+<xacro:include filename="$(find kerby_description)/urdf/materials.xacro" />
+<xacro:include filename="$(find kerby_description)/urdf/kerby.trans" />
+<xacro:include filename="$(find kerby_description)/urdf/kerby.gazebo" />
+<link name="base_link">
+  <inertial>
+    <origin xyz="0.029969421077976243 0.10500332317031125 -0.11062962842827315" rpy="0 0 0"/>
+    <mass value="49.646028993833724"/>
+    <inertia ixx="1.707273" iyy="2.534956" izz="2.455449" ixy="-0.019527" iyz="-0.055493" ixz="-0.42303"/>
+  </inertial>
+  <visual>
+    <origin xyz="0 0 0" rpy="0 0 0"/>
+    <geometry>
+      <mesh filename="package://kerby_description/meshes/base_link.stl" scale="0.001 0.001 0.001"/>
+    </geometry>
+    <material name="blue"/>
+  </visual>
+  <collision>
+    <origin xyz="0 0 0" rpy="0 0 0"/>
+    <geometry>
+      <mesh filename="package://kerby_description/meshes/base_link.stl" scale="0.001 0.001 0.001"/>
+    </geometry>
+  </collision>
+</link>
+<link name="steering_1">
+  <inertial>
+    <origin xyz="0.0029876037310104797 -0.036027674549748256 -0.21327240320670968" rpy="0 0 0"/>
+    <mass value="0.3543584805415501"/>
+    <inertia ixx="0.003568" iyy="0.003121" izz="0.000552" ixy="1.7e-05" iyz="-0.000205" ixz="3.2e-05"/>
+  </inertial>
+  <visual>
+    <origin xyz="-0.423307 -0.476325 0.140943" rpy="0 0 0"/>
+    <geometry>
+      <mesh filename="package://kerby_description/meshes/steering_1.stl" scale="0.001 0.001 0.001"/>
+    </geometry>
+    <material name="silver"/>
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
File: hd_ws/src/control/kerby_moveit_config_ugly/config/kerby.ros2_control.xacro (robot description, xacro)
@@ -7,7 +7,9 @@
                 <!-- By default, set up controllers for simulation. This won't work on real hardware -->
                 <plugin>kerby_hw_interface/KerbyArmInterface</plugin>
+                <!--  gazebo_ros2_control/GazeboSystem    mock_components/GenericSystem   kerby_hw_interface/KerbyArmInterface  -->
             </hardware>
             <joint name="joint1">
                 <command_interface name="position"/>
+                <!-- <command_interface name="velocity"/> -->
                 <state_interface name="position">
                   <param name="initial_value">${initial_positions['joint1']}</param>
@@ -17,4 +19,5 @@
             <joint name="joint2">
                 <command_interface name="position"/>
+                <!-- <command_interface name="velocity"/> -->
                 <state_interface name="position">
                   <param name="initial_value">${initial_positions['joint2']}</param>
@@ -24,4 +27,5 @@
             <joint name="joint3">
                 <command_interface name="position"/>
+                <!-- <command_interface name="velocity"/> -->
                 <state_interface name="position">
                   <param name="initial_value">${initial_positions['joint3']}</param>
@@ -31,4 +35,5 @@
             <joint name="joint4">
                 <command_interface name="position"/>
+                <!-- <command_interface name="velocity"/> -->
                 <state_interface name="position">
                   <param name="initial_value">${initial_positions['joint4']}</param>
@@ -38,4 +43,5 @@
             <joint name="joint5">
                 <command_interface name="position"/>
+                <!-- <command_interface name="velocity"/> -->
                 <state_interface name="position">
                   <param name="initial_value">${initial_positions['joint5']}</param>
@@ -45,4 +51,5 @@
             <joint name="joint6">
                 <command_interface name="position"/>
+                <!-- <command_interface name="velocity"/> -->
                 <state_interface name="position">
                   <param name="initial_value">${initial_positions['joint6']}</param>
@@ -50,5 +57,18 @@
                 <state_interface name="velocity"/>
             </joint>
+            <joint name="gripper_left_finger_joint">
+                <command_interface name="position"/>
+                <!-- <command_interface name="velocity"/> -->
+                <state_interface name="position">
+                  <param name="initial_value">${initial_positions['gripper_left_finger_joint']}</param>
+                </state_interface>
+                <state_interface name="velocity"/>
+            </joint>
         </ros2_control>
+    <gazebo>
+      <plugin name="gazebo_ros2_control" filename="libgazebo_ros2_control.so">
+        <parameters>$(find kerby_moveit_config)/config/ros2_controllers.yaml</parameters>
+      </plugin>
+    </gazebo>
     </xacro:macro>
 </robot>

Commit message: added finger1 to ik

File: hd_ws/src/control/kerby_description/urdf/kerby.urdf.xacro (robot description, xacro)
@@ -495,4 +495,5 @@
   <axis xyz="-0.986688 -0.018348 -0.161587"/>
   <limit upper="0.0" lower="0.0" effort="100" velocity="100"/>
+  <mimic joint="finger1" multiplier="-1" offset="0"/>
 </joint>
 <joint name="moteurJ3" type="fixed">

File: hd_ws/src/control/kerby_moveit_config/config/kerby.ros2_control.xacro (robot description, xacro)
@@ -50,4 +50,11 @@
                 <state_interface name="velocity"/>
             </joint>
+            <joint name="finger1">
+                <command_interface name="position"/>
+                <state_interface name="position">
+                  <param name="initial_value">${initial_positions['finger1']}</param>
+                </state_interface>
+                <state_interface name="velocity"/>
+            </joint>
         </ros2_control>
     </xacro:macro>
