Commit message: cleanup of outdated packages

File: hd_ws/src/control/kerby_description/urdf/kerby.urdf.xacro (robot description, xacro)
@@ -6,5 +6,5 @@
 <link name="base_link">
   <inertial>
-    <origin xyz="0.029969421077976243 0.10500332317031125 -0.11062962842827315" rpy="0 0 0"/>
+    <origin xyz="0.029969421077976347 0.10500332317031078 -0.11062962842827342" rpy="0 0 0"/>
     <mass value="49.646028993833724"/>
     <inertia ixx="1.707273" iyy="2.534956" izz="2.455449" ixy="-0.019527" iyz="-0.055493" ixz="-0.42303"/>
@@ -26,5 +26,5 @@
 <link name="steering_1">
   <inertial>
-    <origin xyz="0.0029876037310104797 -0.036027674549748256 -0.21327240320670968" rpy="0 0 0"/>
+    <origin xyz="0.0029876037310107573 -0.03602767454974787 -0.21327240320670968" rpy="0 0 0"/>
     <mass value="0.3543584805415501"/>
     <inertia ixx="0.003568" iyy="0.003121" izz="0.000552" ixy="1.7e-05" iyz="-0.000205" ixz="3.2e-05"/>
@@ -46,5 +46,5 @@
 <link name="steering_2">
   <inertial>
-    <origin xyz="-0.0029877917009971666 0.03602790788253926 -0.21327245240653883" rpy="0 0 0"/>
+    <origin xyz="-0.0029877917009968336 0.036027907882538956 -0.21327245240653972" rpy="0 0 0"/>
     <mass value="0.3543584805415501"/>
     <inertia ixx="0.003568" iyy="0.003121" izz="0.000552" ixy="1.7e-05" iyz="0.000205" ixz="-3.2e-05"/>
@@ -66,5 +66,5 @@
 <link name="steering_3">
   <inertial>
-    <origin xyz="-0.0029882539688567133 0.03602790788253865 -0.21327240320671673" rpy="0 0 0"/>
+    <origin xyz="-0.0029882539688568244 0.03602790788253865 -0.21327240320671773" rpy="0 0 0"/>
     <mass value="0.3543584805415501"/>
     <inertia ixx="0.003568" iyy="0.003121" izz="0.000552" ixy="1.7e-05" iyz="0.000205" ixz="-3.2e-05"/>
@@ -86,5 +86,5 @@
 <link name="steering_4">
   <inertial>
-    <origin xyz="0.0029881414631521275 -0.03602767454974787 -0.2132724524065319" rpy="0 0 0"/>
+    <origin xyz="0.002988141463151961 -0.03602767454974776 -0.21327245240653173" rpy="0 0 0"/>
     <mass value="0.3543584805415501"/>
     <inertia ixx="0.003568" iyy="0.003121" izz="0.000552" ixy="1.7e-05" iyz="-0.000205" ixz="3.2e-05"/>
@@ -106,5 +106,5 @@
 <link name="wheel3_1">
   <inertial>
-    <origin xyz="0.0003400707098370481 -0.010197254794898913 3.6630334474541115e-06" rpy="0 0 0"/>
+    <origin xyz="0.0003400707098368816 -0.010197254794898913 3.6630334477316673e-06" rpy="0 0 0"/>
     <mass value="1.592763813314383"/>
     <inertia ixx="0.010896" iyy="0.018605" izz="0.010887" ixy="-0.000257" iyz="-2e-06" ixz="0.0"/>
@@ -126,5 +126,5 @@
 <link name="wheel4_1">
   <inertial>
-    <origin xyz="0.00034053297769459645 -0.010197254794899857 3.712233269614895e-06" rpy="0 0 0"/>
+    <origin xyz="0.0003405329776948185 -0.010197254794899857 3.712233269614895e-06" rpy="0 0 0"/>
     <mass value="1.592763813314383"/>
     <inertia ixx="0.010896" iyy="0.018605" izz="0.010887" ixy="-0.000257" iyz="-2e-06" ixz="0.0"/>
@@ -146,5 +146,5 @@
 <link name="wheel2_1">
   <inertial>
-    <origin xyz="-0.0003401832155410234 0.010196488127690972 3.712233261510267e-06" rpy="0 0 0"/>
+    <origin xyz="-0.0003401832155410234 0.010196488127690917 3.712233260733111e-06" rpy="0 0 0"/>
     <mass value="1.592763813314383"/>
     <inertia ixx="0.010896" iyy="0.018605" izz="0.010887" ixy="-0.000257" iyz="2e-06" ixz="-0.0"/>
@@ -166,5 +166,5 @@
 <link name="wheel1_1">
   <inertial>
-    <origin xyz="-0.00033972094768197625 0.010196488127692027 3.6630334394605057e-06" rpy="0 0 0"/>
+    <origin xyz="-0.0003397209476816987 0.010196488127692138 3.6630334383502827e-06" rpy="0 0 0"/>
     <mass value="1.592763813314383"/>
     <inertia ixx="0.010896" iyy="0.018605" izz="0.010887" ixy="-0.000257" iyz="2e-06" ixz="-0.0"/>
@@ -186,7 +186,7 @@
 <link name="hd_link2_1">
   <inertial>
-    <origin xyz="-0.06551545688031782 0.0608390658028839 0.12833264938052846" rpy="0 0 0"/>
+    <origin xyz="0.0033070766839577714 0.06083906580288365 0.1440505220890836" rpy="0 0 0"/>
     <mass value="2.4452075265656514"/>
-    <inertia ixx="0.0307" iyy="0.03827" izz="0.011048" ixy="-0.000736" iyz="0.001431" ixz="0.01488"/>
+    <inertia ixx="0.038706" iyy="0.03827" izz="0.003043" ixy="3.2e-05" iyz="0.001609" ixz="-5e-05"/>
   </inertial>
   <visual>
@@ -206,10 +206,10 @@
 <link name="hd_link3_1">
   <inertial>
-    <origin xyz="-0.18835718544023639 -0.028188435052669616 0.002484829044890391" rpy="0 0 0"/>
+    <origin xyz="-0.18542255123016124 -0.02818843505267088 0.033215191672649136" rpy="0 0 0"/>
     <mass value="0.3993227194340243"/>
-    <inertia ixx="0.000928" iyy="0.00625" izz="0.006285" ixy="4.5e-05" iyz="3e-06" ixz="-0.000722"/>
-  </inertial>
-  <visual>
-    <origin xyz="0.418083 -0.132217 -0.398623" rpy="0 0 0"/>
+    <inertia ixx="0.000838" iyy="0.00625" izz="0.006374" ixy="4.5e-05" iyz="-5e-06" ixz="0.00018"/>
+  </inertial>
+  <visual>
+    <origin xyz="0.22795 -0.132217 -0.446313" rpy="0 0 0"/>
     <geometry>
       <mesh filename="package://kerby_description/meshes/hd_link3_1.stl" scale="0.001 0.001 0.001"/>
@@ -218,5 +218,5 @@
   </visual>
   <collision>
-    <origin xyz="0.418083 -0.132217 -0.398623" rpy="0 0 0"/>
+    <origin xyz="0.22795 -0.132217 -0.446313" rpy="0 0 0"/>
     <geometry>
       <mesh filename="package://kerby_description/meshes/hd_link3_1.stl" scale="0.001 0.001 0.001"/>
@@ -226,10 +226,10 @@
 <link name="hd_link4_1">
   <inertial>
-    <origin xyz="-0.02605467768013403 0.0028968395456621804 -0.00492049213285306" rpy="0 0 0"/>
+    <origin xyz="-0.026508760059289482 0.0028968395456604734 -0.000598737646716252" rpy="0 0 0"/>
     <mass value="0.16590781468918114"/>
-    <inertia ixx="0.000204" iyy="0.000349" izz="0.000469" ixy="3.8e-05" iyz="1.2e-05" ixz="-4.4e-05"/>
-  </inertial>
-  <visual>
-    <origin xyz="0.734928 -0.102573 -0.381483" rpy="0 0 0"/>
+    <inertia ixx="0.000197" iyy="0.000349" izz="0.000476" ixy="3.9e-05" iyz="5e-06" ixz="1e-06"/>
+  </inertial>
+  <visual>
+    <origin xyz="0.54334 -0.102573 -0.481152" rpy="0 0 0"/>
     <geometry>
       <mesh filename="package://kerby_description/meshes/hd_link4_1.stl" scale="0.001 0.001 0.001"/>
@@ -238,5 +238,5 @@
   </visual>
   <collision>
-    <origin xyz="0.734928 -0.102573 -0.381483" rpy="0 0 0"/>
+    <origin xyz="0.54334 -0.102573 -0.481152" rpy="0 0 0"/>
     <geometry>
       <mesh filename="package://kerby_description/meshes/hd_link4_1.stl" scale="0.001 0.001 0.001"/>
@@ -246,10 +246,10 @@
 <link name="hd_link5_1">
   <inertial>
-    <origin xyz="0.0006595883387678914 0.03846053744230657 -0.0032042955275293217" rpy="0 0 0"/>
-    <mass value="0.06877842327462745"/>
-    <inertia ixx="4.3e-05" iyy="2.9e-05" izz="4.9e-05" ixy="-0.0" iyz="1e-06" ixz="-1e-06"/>
-  </inertial>
-  <visual>
-    <origin xyz="0.827396 -0.060573 -0.36634" rpy="0 0 0"/>
+    <origin xyz="-0.00326876427210665 0.038460537452552596 -0.0001281048652070904" rpy="0 0 0"/>
+    <mass value="0.06877842327462741"/>
+    <inertia ixx="4.9e-05" iyy="2.9e-05" izz="4.3e-05" ixy="1e-06" iyz="0.0" ixz="0.0"/>
+  </inertial>
+  <visual>
+    <origin xyz="0.63704 -0.060573 -0.481315" rpy="0 0 0"/>
     <geometry>
       <mesh filename="package://kerby_description/meshes/hd_link5_1.stl" scale="0.001 0.001 0.001"/>
@@ -258,5 +258,5 @@
   </visual>
   <collision>
-    <origin xyz="0.827396 -0.060573 -0.36634" rpy="0 0 0"/>
+    <origin xyz="0.63704 -0.060573 -0.481315" rpy="0 0 0"/>
     <geometry>
       <mesh filename="package://kerby_description/meshes/hd_link5_1.stl" scale="0.001 0.001 0.001"/>
@@ -266,10 +266,10 @@
 <link name="hd_link6_1">
   <inertial>
-    <origin xyz="0.006667844950576041 -0.0007677997590191804 -0.03456780245146873" rpy="0 0 0"/>
+    <origin xyz="-0.03520188089997378 -0.0007184800362615151 0.000553267969914728" rpy="0 0 0"/>
     <mass value="0.11153016933793788"/>
-    <inertia ixx="0.000164" iyy="0.000263" izz="0.000119" ixy="-1e-06" iyz="-0.0" ixz="1e-05"/>
-  </inertial>
-  <visual>
-    <origin xyz="0.822824 -0.102533 -0.339729" rpy="0 0 0"/>
+    <inertia ixx="0.000117" iyy="0.000166" izz="0.000263" ixy="-2e-06" iyz="-1e-06" ixz="-1e-06"/>
+  </inertial>
+  <visual>
+    <origin xyz="0.66404 -0.102533 -0.48115" rpy="0 0 0"/>
     <geometry>
       <mesh filename="package://kerby_description/meshes/hd_link6_1.stl" scale="0.001 0.001 0.001"/>
@@ -278,5 +278,5 @@
   </visual>
   <collision>
-    <origin xyz="0.822824 -0.102533 -0.339729" rpy="0 0 0"/>
+    <origin xyz="0.66404 -0.102533 -0.48115" rpy="0 0 0"/>
     <geometry>
       <mesh filename="package://kerby_description/meshes/hd_link6_1.stl" scale="0.001 0.001 0.001"/>
@@ -286,10 +286,10 @@
 <link name="hd_finger2_1">
   <inertial>
-    <origin xyz="0.7203862006849536 0.09659828189006314 0.26002341296854425" rpy="0 0 0"/>
+    <origin xyz="0.36572155404860496 -0.7471770274512002 -0.09385171158022082" rpy="0 0 0"/>
     <mass value="0.025342855198124774"/>
-    <inertia ixx="1.7e-05" iyy="1.6e-05" izz="5e-06" ixy="-1e-06" iyz="2e-06" ixz="4e-06"/>
-  </inertial>
-  <visual>
-    <origin xyz="1.574668 -0.00212 0.029503" rpy="0 0 0"/>
+    <inertia ixx="4e-06" iyy="1.8e-05" izz="1.6e-05" ixy="-2e-06" iyz="-0.0" ixz="-2e-06"/>
+  </inertial>
+  <visual>
+    <origin xyz="1.132411 -0.857299 -0.577422" rpy="0 0 0"/>
     <geometry>
       <mesh filename="package://kerby_description/meshes/hd_finger2_1.stl" scale="0.001 0.001 0.001"/>
@@ -298,5 +298,5 @@
   </visual>
   <collision>
-    <origin xyz="1.574668 -0.00212 0.029503" rpy="0 0 0"/>
+    <origin xyz="1.132411 -0.857299 -0.577422" rpy="0 0 0"/>
     <geometry>
       <mesh filename="package://kerby_description/meshes/hd_finger2_1.stl" scale="0.001 0.001 0.001"/>
@@ -306,10 +306,10 @@
 <link name="hd_finger1_1">
   <inertial>
-    <origin xyz="0.8454061278845124 0.12710568875536565 0.27256760789282636" rpy="0 0 0"/>
+    <origin xyz="0.34237822893598846 -0.7617001148724551 -0.1442671674369853" rpy="0 0 0"/>
     <mass value="0.025342855198124774"/>
-    <inertia ixx="1.8e-05" iyy="1.6e-05" izz="4e-06" ixy="0.0" iyz="-2e-06" ixz="1e-06"/>
-  </inertial>
-  <visual>
-    <origin xyz="1.618854 0.021073 0.029157" rpy="0 0 0"/>
+    <inertia ixx="4e-06" iyy="1.8e-05" izz="1.6e-05" ixy="2e-06" iyz="-0.0" ixz="2e-06"/>
+  </inertial>
+  <visual>
+    <origin xyz="1.10949 -0.856977 -0.62175" rpy="0 0 0"/>
     <geometry>
       <mesh filename="package://kerby_description/meshes/hd_finger1_1.stl" scale="0.001 0.001 0.001"/>
@@ -318,5 +318,5 @@
   </visual>
   <collision>
-    <origin xyz="1.618854 0.021073 0.029157" rpy="0 0 0"/>
+    <origin xyz="1.10949 -0.856977 -0.62175" rpy="0 0 0"/>
     <geometry>
       <mesh filename="package://kerby_description/meshes/hd_finger1_1.stl" scale="0.001 0.001 0.001"/>
@@ -326,10 +326,10 @@
 <link name="hd_motor_j3_1">
   <inertial>
-    <origin xyz="-0.2875958225986405 0.29755094640210267 -0.017659454596450352" rpy="0 0 0"/>
+    <origin xyz="-0.26883632684956255 0.15032394640210167 0.12504846034721717" rpy="0 0 0"/>
     <mass value="0.11925838600046076"/>
-    <inertia ixx="0.000465" iyy="0.000525" izz="7.4e-05" ixy="0.0" iyz="-0.0" ixz="0.000165"/>
-  </inertial>
-  <visual>
-    <origin xyz="-0.008356 0.196334 -0.326442" rpy="0 0 0"/>
+    <inertia ixx="0.000514" iyy="0.000525" izz="2.4e-05" ixy="-0.0" iyz="-0.0" ixz="-7.3e-05"/>
+  </inertial>
+  <visual>
+    <origin xyz="-0.12039 0.049107 -0.176255" rpy="0 0 0"/>
     <geometry>
       <mesh filename="package://kerby_description/meshes/hd_motor_j3_1.stl" scale="0.001 0.001 0.001"/>
@@ -338,5 +338,5 @@
   </visual>
   <collision>
-    <origin xyz="-0.008356 0.196334 -0.326442" rpy="0 0 0"/>
+    <origin xyz="-0.12039 0.049107 -0.176255" rpy="0 0 0"/>
     <geometry>
       <mesh filename="package://kerby_description/meshes/hd_motor_j3_1.stl" scale="0.001 0.001 0.001"/>
@@ -346,5 +346,5 @@
 <link name="pivot_droit_1">
   <inertial>
-    <origin xyz="3.14351229217932e-05 0.11623514902532228 0.01341038188021934" rpy="0 0 0"/>
+    <origin xyz="3.143512292182876e-05 0.11623514902532184 0.013410381880219507" rpy="0 0 0"/>
     <mass value="1.6615144825592312"/>
     <inertia ixx="0.006305" iyy="0.220618" izz="0.221436" ixy="1e-06" iyz="-0.000817" ixz="-0.001791"/>
@@ -366,5 +366,5 @@
 <link name="hd_link1_1">
   <inertial>
-    <origin xyz="0.0001907779404473342 0.014210553405146945 0.03342137346722488" rpy="0 0 0"/>
+    <origin xyz="0.00019077794044744523 0.01421055340514632 0.03342137346722458" rpy="0 0 0"/>
     <mass value="0.3391136619658369"/>
     <inertia ixx="0.001801" iyy="0.001217" izz="0.00078" ixy="1e-05" iyz="-0.000142" ixz="-8e-06"/>
@@ -386,5 +386,5 @@
 <link name="pivot_gauche_1">
   <inertial>
-    <origin xyz="-3.208536076750555e-05 -0.1162349156925368 0.01341038188021211" rpy="0 0 0"/>
+    <origin xyz="-3.2085360767372846e-05 -0.11623491569253713 0.013410381880211292" rpy="0 0 0"/>
     <mass value="1.6615144825592312"/>
     <inertia ixx="0.006305" iyy="0.220618" izz="0.221436" ixy="1e-06" iyz="0.000817" ixz="0.001791"/>
@@ -459,5 +459,5 @@
 </joint>
 <joint name="joint3" type="continuous">
-  <origin xyz="-0.18944 0.088 0.352405" rpy="0 0 0"/>
+  <origin xyz="0.000693 0.088 0.400095" rpy="0 0 0"/>
   <parent link="hd_link2_1"/>
   <child link="hd_link3_1"/>
@@ -465,38 +465,38 @@
 </joint>
 <joint name="joint4" type="continuous">
-  <origin xyz="-0.316845 -0.029644 -0.01714" rpy="0 0 0"/>
+  <origin xyz="-0.31539 -0.029644 0.034839" rpy="0 0 0"/>
   <parent link="hd_link3_1"/>
   <child link="hd_link4_1"/>
-  <axis xyz="0.986854 0.0 0.161617"/>
+  <axis xyz="0.999999 0.0 -0.001732"/>
 </joint>
 <joint name="joint5" type="continuous">
-  <origin xyz="-0.092468 -0.042 -0.015143" rpy="0 0 0"/>
+  <origin xyz="-0.0937 -0.042 0.000163" rpy="0 0 0"/>
   <parent link="hd_link4_1"/>
   <child link="hd_link5_1"/>
-  <axis xyz="-0.0 -1.0 0.0"/>
+  <axis xyz="0.0 -1.0 0.0"/>
 </joint>
 <joint name="joint6" type="continuous">
-  <origin xyz="0.004572 0.04196 -0.026611" rpy="0 0 0"/>
+  <origin xyz="-0.027 0.04196 -0.000165" rpy="0 0 0"/>
   <parent link="hd_link5_1"/>
   <child link="hd_link6_1"/>
-  <axis xyz="0.169333 -0.0 -0.985559"/>
+  <axis xyz="-0.999981 -0.0 -0.006092"/>
 </joint>
 <joint name="finger1" type="prismatic">
-  <origin xyz="-0.751844 -0.100413 -0.369232" rpy="0 0 0"/>
+  <origin xyz="-0.468371 0.754766 0.096272" rpy="0 0 0"/>
   <parent link="hd_link6_1"/>
   <child link="hd_finger2_1"/>
-  <axis xyz="-0.986688 -0.018348 -0.161587"/>
+  <axis xyz="0.007713 0.999801 0.018395"/>
   <limit upper="0.0" lower="0.0" effort="100" velocity="100"/>
 </joint>
 <joint name="finger2" type="prismatic">
-  <origin xyz="-0.79603 -0.123606 -0.368886" rpy="0 0 0"/>
+  <origin xyz="-0.44545 0.754444 0.1406" rpy="0 0 0"/>
   <parent link="hd_link6_1"/>
   <child link="hd_finger1_1"/>
-  <axis xyz="-0.986688 -0.018348 -0.161587"/>
+  <axis xyz="0.007713 0.999801 0.018395"/>
   <limit upper="0.0" lower="0.0" effort="100" velocity="100"/>
   <mimic joint="finger1" multiplier="-1" offset="0"/>
 </joint>
 <joint name="moteurJ3" type="fixed">
-  <origin xyz="0.236999 -0.240551 0.280224" rpy="0 0 0"/>
+  <origin xyz="0.349033 -0.093324 0.130037" rpy="0 0 0"/>
   <parent link="hd_link2_1"/>
   <child link="hd_motor_j3_1"/>

File: hd_ws/src/control/kerby_moveit_config/config/kerby.urdf.xacro (robot description, xacro)
@@ -3,5 +3,5 @@
     <xacro:arg name="initial_positions_file" default="initial_positions.yaml" />
     <!-- Import kerby urdf file -->
-    <xacro:include filename="$(find Assemblage_description)/urdf/Assemblage.urdf.xacro" />
+    <xacro:include filename="$(find kerby_description)/urdf/kerby.urdf.xacro" />
     <!-- Import control_xacro -->
     <xacro:include filename="kerby.ros2_control.xacro" />

Commit message: velocity limits set for moveit

File: hd_ws/src/control/kerby_description/urdf/kerby.urdf.xacro (robot description, xacro)
@@ -4,4 +4,26 @@
 <xacro:include filename="$(find kerby_description)/urdf/kerby.trans" />
 <xacro:include filename="$(find kerby_description)/urdf/kerby.gazebo" />
+<xacro:property name="rpm_to_Radps" value="${2*pi/60.0}" />     <!-- rotations per minute to Rad per second conversion -->
+<xacro:macro name="aaa_joint_limits" params="lower:=0.0 upper:=0.0 velocity:=${rpm_to_Radps} effort:=100.0">
+  <limit lower="${lower}" upper="${upper}" velocity="${velocity}" effort="${effort}"/>
+</xacro:macro>
+<xacro:property name="joint1_limits">
+  <xacro:aaa_joint_limits lower="${-pi}" upper="${pi}" velocity="${0.5*rpm_to_Radps}" />
+</xacro:property>
+<xacro:property name="joint2_limits">
+  <xacro:aaa_joint_limits lower="${-pi/30}" upper="${pi/30}" velocity="${0.5*rpm_to_Radps}" />
+</xacro:property>
+<xacro:property name="joint3_limits">
+  <xacro:aaa_joint_limits lower="${-pi/4}" upper="${pi/4}" velocity="${1*rpm_to_Radps}" />
+</xacro:property>
+<xacro:property name="joint4_limits">
+  <xacro:aaa_joint_limits lower="${-pi}" upper="${pi}" velocity="${2*rpm_to_Radps}" />
+</xacro:property>
+<xacro:property name="joint5_limits">
+  <xacro:aaa_joint_limits lower="${-pi/4}" upper="${pi/4}" velocity="${1.5*rpm_to_Radps}" />
+</xacro:property>
+<xacro:property name="joint6_limits">
+  <xacro:aaa_joint_limits lower="${-pi/2}" upper="${pi/2}" velocity="${2*rpm_to_Radps}" />
+</xacro:property>
 <link name="base_link">
   <inertial>
@@ -457,4 +479,5 @@
   <child link="hd_link2_1"/>
   <axis xyz="0.0 1.0 0.0"/>
+  <xacro:insert_block name="joint2_limits" />
 </joint>
 <joint name="joint3" type="continuous">
@@ -463,4 +486,5 @@
   <child link="hd_link3_1"/>
   <axis xyz="-0.0 1.0 0.0"/>
+  <xacro:insert_block name="joint3_limits" />
 </joint>
 <joint name="joint4" type="continuous">
@@ -469,4 +493,5 @@
   <child link="hd_link4_1"/>
   <axis xyz="0.999999 0.0 -0.001732"/>
+  <xacro:insert_block name="joint4_limits" />
 </joint>
 <joint name="joint5" type="continuous">
@@ -475,4 +500,5 @@
   <child link="hd_link5_1"/>
   <axis xyz="0.0 -1.0 0.0"/>
+  <xacro:insert_block name="joint5_limits" />
 </joint>
 <joint name="joint6" type="continuous">
@@ -481,4 +507,5 @@
   <child link="hd_link6_1"/>
   <axis xyz="-0.999981 -0.0 -0.006092"/>
+  <xacro:insert_block name="joint6_limits" />
 </joint>
 <joint name="finger1" type="prismatic">
@@ -513,4 +540,6 @@
   <child link="hd_link1_1"/>
   <axis xyz="0.0 -0.0 1.0"/>
+  <xacro:insert_block name="joint1_limits" />
+  <!-- <limit lower="${-pi}" upper="${pi}" velocity="${2*rpm_to_Radps}" effort="100" /> -->
 </joint>
 <joint name="pivot_droit" type="continuous">

Commit message: mash

File: hd_ws/src/control/kerby_description/urdf/kerby.urdf.xacro (robot description, xacro)
@@ -5,24 +5,25 @@
 <xacro:include filename="$(find kerby_description)/urdf/kerby.gazebo" />
 <xacro:property name="rpm_to_Radps" value="${2*pi/60.0}" />     <!-- rotations per minute to Rad per second conversion -->
+<xacro:property name="velocity_scaling" value="1.0" />     <!-- allows to scale all max velocities down at once -->
 <xacro:macro name="aaa_joint_limits" params="lower:=0.0 upper:=0.0 velocity:=${rpm_to_Radps} effort:=100.0">
   <limit lower="${lower}" upper="${upper}" velocity="${velocity}" effort="${effort}"/>
 </xacro:macro>
 <xacro:property name="joint1_limits">
-  <xacro:aaa_joint_limits lower="${-100*pi}" upper="${100*pi}" velocity="${2 * rpm_to_Radps}" />
+  <xacro:aaa_joint_limits lower="${-pi}" upper="${pi}" velocity="${2 * rpm_to_Radps * velocity_scaling}" />
 </xacro:property>
 <xacro:property name="joint2_limits">
-  <xacro:aaa_joint_limits lower="${-100*pi/30}" upper="${100*pi/30}" velocity="${1.5 * rpm_to_Radps}" />
+  <xacro:aaa_joint_limits lower="${-pi/2}" upper="${pi/2}" velocity="${1.5 * rpm_to_Radps * velocity_scaling}" />
 </xacro:property>
 <xacro:property name="joint3_limits">
-  <xacro:aaa_joint_limits lower="${-100*pi/4}" upper="${100*pi/4}" velocity="${1.5 * rpm_to_Radps}" />
+  <xacro:aaa_joint_limits lower="${-pi/4}" upper="${pi/4}" velocity="${1.5 * rpm_to_Radps * velocity_scaling}" />
 </xacro:property>
 <xacro:property name="joint4_limits">
-  <xacro:aaa_joint_limits lower="${-100*pi}" upper="${100*pi}" velocity="${6 * rpm_to_Radps}" />
+  <xacro:aaa_joint_limits lower="${-1.5*pi}" upper="${1.5*pi}" velocity="${6 * rpm_to_Radps * velocity_scaling}" />
 </xacro:property>
 <xacro:property name="joint5_limits">
-  <xacro:aaa_joint_limits lower="${-100*pi/4}" upper="${100*pi/4}" velocity="${2 * rpm_to_Radps}" />
+  <xacro:aaa_joint_limits lower="${-pi/2}" upper="${pi/2}" velocity="${2 * rpm_to_Radps * velocity_scaling}" />
 </xacro:property>
 <xacro:property name="joint6_limits">
-  <xacro:aaa_joint_limits lower="${-100*pi/2}" upper="${100*pi/2}" velocity="${6 * rpm_to_Radps}" />
+  <xacro:aaa_joint_limits lower="${-pi}" upper="${pi}" velocity="${6 * rpm_to_Radps * velocity_scaling}" />
 </xacro:property>
 <link name="base_link">
@@ -474,5 +475,5 @@
   <axis xyz="0.033329 -0.999444 -0.000279"/>
 </joint>
-<joint name="joint2" type="continuous">
+<joint name="joint2" type="revolute">
   <origin xyz="0.0 -0.0577 0.102" rpy="0 0 0"/>
   <parent link="hd_link1_1"/>
@@ -481,5 +482,5 @@
   <xacro:insert_block name="joint2_limits" />
 </joint>
-<joint name="joint3" type="continuous">
+<joint name="joint3" type="revolute">
   <origin xyz="0.000693 0.088 0.400095" rpy="0 0 0"/>
   <parent link="hd_link2_1"/>
@@ -488,5 +489,5 @@
   <xacro:insert_block name="joint3_limits" />
 </joint>
-<joint name="joint4" type="continuous">
+<joint name="joint4" type="revolute">
   <origin xyz="-0.31539 -0.029644 0.034839" rpy="0 0 0"/>
   <parent link="hd_link3_1"/>
@@ -495,5 +496,5 @@
   <xacro:insert_block name="joint4_limits" />
 </joint>
-<joint name="joint5" type="continuous">
+<joint name="joint5" type="revolute">
   <origin xyz="-0.0937 -0.042 0.000163" rpy="0 0 0"/>
   <parent link="hd_link4_1"/>
@@ -502,5 +503,5 @@
   <xacro:insert_block name="joint5_limits" />
 </joint>
-<joint name="joint6" type="continuous">
+<joint name="joint6" type="revolute">
   <origin xyz="-0.027 0.04196 -0.000165" rpy="0 0 0"/>
   <parent link="hd_link5_1"/>
@@ -535,5 +536,5 @@
   <axis xyz="0.0 -1.0 -0.0"/>
 </joint>
-<joint name="joint1" type="continuous">
+<joint name="joint1" type="revolute">
   <origin xyz="-0.228643 0.101917 -0.055782" rpy="0 0 0"/>
   <parent link="base_link"/>
