Commit message: new from foxy branch

File: hd_ws/src/control/Assemblage_description/urdf/Assemblage.urdf.xacro (robot description, xacro)
@@ -1,12 +1,35 @@
 <?xml version="1.0" ?>
-<robot name="Assemblage" xmlns:xacro="http://www.ros.org/wiki/xacro">
+<robot name="kerby" xmlns:xacro="http://www.ros.org/wiki/xacro">
 <xacro:include filename="$(find Assemblage_description)/urdf/materials.xacro" />
 <xacro:include filename="$(find Assemblage_description)/urdf/Assemblage.trans" />
 <xacro:include filename="$(find Assemblage_description)/urdf/Assemblage.gazebo" />
+<xacro:property name="rpm_to_Radps" value="${2*pi/60.0}" />     <!-- rotations per minute to Rad per second conversion -->
+<xacro:property name="velocity_scaling" value="1.0" />     <!-- allows to scale all max velocities down at once -->
+<xacro:macro name="aaa_joint_limits" params="lower:=0.0 upper:=0.0 velocity:=${rpm_to_Radps} effort:=100.0">
+  <limit lower="${lower}" upper="${upper}" velocity="${velocity}" effort="${effort}"/>
+</xacro:macro>
+<xacro:property name="joint1_limits">
+  <xacro:aaa_joint_limits lower="${-1.5*pi}" upper="${1.5*pi}" velocity="${3 * rpm_to_Radps * velocity_scaling}" />
+</xacro:property>
+<xacro:property name="joint2_limits">
+  <xacro:aaa_joint_limits lower="${-pi}" upper="${pi/2}" velocity="${1 * rpm_to_Radps * velocity_scaling}" />
+</xacro:property>
+<xacro:property name="joint3_limits">
+  <xacro:aaa_joint_limits lower="${-pi/4}" upper="${pi/4}" velocity="${1.5 * rpm_to_Radps * velocity_scaling}" />
+</xacro:property>
+<xacro:property name="joint4_limits">
+  <xacro:aaa_joint_limits lower="${-2*pi}" upper="${2*pi}" velocity="${6 * rpm_to_Radps * velocity_scaling}" />
+</xacro:property>
+<xacro:property name="joint5_limits">
+  <xacro:aaa_joint_limits lower="${-pi/2}" upper="${pi/2}" velocity="${2 * rpm_to_Radps * velocity_scaling}" />
+</xacro:property>
+<xacro:property name="joint6_limits">
+  <xacro:aaa_joint_limits lower="${-pi}" upper="${pi}" velocity="${6 * rpm_to_Radps * velocity_scaling}" />
+</xacro:property>
 <link name="base_link">
   <inertial>
-    <origin xyz="0.029969421077976347 0.10500332317031078 -0.11062962842827342" rpy="0 0 0"/>
-    <mass value="49.646028993833724"/>
-    <inertia ixx="1.707273" iyy="2.534956" izz="2.455449" ixy="-0.019527" iyz="-0.055493" ixz="-0.42303"/>
+    <origin xyz="0.05362398614035063 0.01974617698532859 0.037120813316089823" rpy="0 0 0"/>
+    <mass value="6.257043020156179"/>
+    <inertia ixx="0.340644" iyy="0.466541" izz="0.402706" ixy="0.000337" iyz="0.00055" ixz="-0.092411"/>
   </inertial>
   <visual>
@@ -26,10 +49,10 @@
 <link name="steering_1">
   <inertial>
-    <origin xyz="0.0029876037310107573 -0.03602767454974787 -0.21327240320670968" rpy="0 0 0"/>
+    <origin xyz="-0.01189644601781037 -0.036027929982466456 -0.2129618322901442" rpy="0 0 0"/>
     <mass value="0.3543584805415501"/>
-    <inertia ixx="0.003568" iyy="0.003121" izz="0.000552" ixy="1.7e-05" iyz="-0.000205" ixz="3.2e-05"/>
-  </inertial>
-  <visual>
-    <origin xyz="-0.423307 -0.476325 0.140943" rpy="0 0 0"/>
+    <inertia ixx="0.003558" iyy="0.003121" izz="0.000562" ixy="2e-06" iyz="-0.000206" ixz="-0.000178"/>
+  </inertial>
+  <visual>
+    <origin xyz="-0.421384 -0.393882 0.063562" rpy="0 0 0"/>
     <geometry>
       <mesh filename="package://Assemblage_description/meshes/steering_1.stl" scale="0.001 0.001 0.001"/>
@@ -38,5 +61,5 @@
   </visual>
   <collision>
-    <origin xyz="-0.423307 -0.476325 0.140943" rpy="0 0 0"/>
+    <origin xyz="-0.421384 -0.393882 0.063562" rpy="0 0 0"/>
     <geometry>
       <mesh filename="package://Assemblage_description/meshes/steering_1.stl" scale="0.001 0.001 0.001"/>
@@ -46,10 +69,10 @@
 <link name="steering_2">
   <inertial>
-    <origin xyz="-0.0029877917009968336 0.036027907882538956 -0.21327245240653972" rpy="0 0 0"/>
+    <origin xyz="0.011896575272170529 0.03602765244982159 -0.21296112839152875" rpy="0 0 0"/>
     <mass value="0.3543584805415501"/>
-    <inertia ixx="0.003568" iyy="0.003121" izz="0.000552" ixy="1.7e-05" iyz="0.000205" ixz="-3.2e-05"/>
-  </inertial>
-  <visual>
-    <origin xyz="-0.42303 0.272491 0.147921" rpy="0 0 0"/>
+    <inertia ixx="0.003558" iyy="0.003121" izz="0.000562" ixy="2e-06" iyz="0.000206" ixz="0.000178"/>
+  </inertial>
+  <visual>
+    <origin xyz="-0.42341 0.353934 0.012408" rpy="0 0 0"/>
     <geometry>
       <mesh filename="package://Assemblage_description/meshes/steering_2.stl" scale="0.001 0.001 0.001"/>
@@ -58,5 +81,5 @@
   </visual>
   <collision>
-    <origin xyz="-0.42303 0.272491 0.147921" rpy="0 0 0"/>
+    <origin xyz="-0.42341 0.353934 0.012408" rpy="0 0 0"/>
     <geometry>
       <mesh filename="package://Assemblage_description/meshes/steering_2.stl" scale="0.001 0.001 0.001"/>
@@ -66,10 +89,10 @@
 <link name="steering_3">
   <inertial>
-    <origin xyz="-0.0029882539688568244 0.03602790788253865 -0.21327240320671773" rpy="0 0 0"/>
+    <origin xyz="0.011896795779964109 0.03602765244982109 -0.21296183229014454" rpy="0 0 0"/>
     <mass value="0.3543584805415501"/>
-    <inertia ixx="0.003568" iyy="0.003121" izz="0.000552" ixy="1.7e-05" iyz="0.000205" ixz="-3.2e-05"/>
-  </inertial>
-  <visual>
-    <origin xyz="0.410093 0.272491 0.140943" rpy="0 0 0"/>
+    <inertia ixx="0.003558" iyy="0.003121" izz="0.000562" ixy="2e-06" iyz="0.000206" ixz="0.000178"/>
+  </inertial>
+  <visual>
+    <origin xyz="0.408171 0.353934 0.063562" rpy="0 0 0"/>
     <geometry>
       <mesh filename="package://Assemblage_description/meshes/steering_3.stl" scale="0.001 0.001 0.001"/>
@@ -78,5 +101,5 @@
   </visual>
   <collision>
-    <origin xyz="0.410093 0.272491 0.140943" rpy="0 0 0"/>
+    <origin xyz="0.408171 0.353934 0.063562" rpy="0 0 0"/>
     <geometry>
       <mesh filename="package://Assemblage_description/meshes/steering_3.stl" scale="0.001 0.001 0.001"/>
@@ -86,10 +109,10 @@
 <link name="steering_4">
   <inertial>
-    <origin xyz="0.002988141463151961 -0.03602767454974776 -0.21327245240653173" rpy="0 0 0"/>
+    <origin xyz="-0.011896225510015512 -0.036027929982466234 -0.21296112839152861" rpy="0 0 0"/>
     <mass value="0.3543584805415501"/>
-    <inertia ixx="0.003568" iyy="0.003121" izz="0.000552" ixy="1.7e-05" iyz="-0.000205" ixz="3.2e-05"/>
-  </inertial>
-  <visual>
-    <origin xyz="0.409817 -0.476325 0.147921" rpy="0 0 0"/>
+    <inertia ixx="0.003558" iyy="0.003121" izz="0.000562" ixy="2e-06" iyz="-0.000206" ixz="-0.000178"/>
+  </inertial>
+  <visual>
+    <origin xyz="0.410197 -0.393882 0.012408" rpy="0 0 0"/>
     <geometry>
       <mesh filename="package://Assemblage_description/meshes/steering_4.stl" scale="0.001 0.001 0.001"/>
@@ -98,5 +121,5 @@
   </visual>
   <collision>
-    <origin xyz="0.409817 -0.476325 0.147921" rpy="0 0 0"/>
+    <origin xyz="0.410197 -0.393882 0.012408" rpy="0 0 0"/>
     <geometry>
       <mesh filename="package://Assemblage_description/meshes/steering_4.stl" scale="0.001 0.001 0.001"/>
@@ -106,10 +129,10 @@
 <link name="wheel3_1">
   <inertial>
-    <origin xyz="0.0003400707098368816 -0.010197254794898913 3.6630334477316673e-06" rpy="0 0 0"/>
+    <origin xyz="0.0003394916280188287 -0.010196510227617639 -2.006330920018007e-05" rpy="0 0 0"/>
     <mass value="1.592763813314383"/>
-    <inertia ixx="0.010896" iyy="0.018605" izz="0.010887" ixy="-0.000257" iyz="-2e-06" ixz="0.0"/>
-  </inertial>
-  <visual>
-    <origin xyz="0.408112 -0.493016 0.417916" rpy="0 0 0"/>
+    <inertia ixx="0.010896" iyy="0.018605" izz="0.010887" ixy="-0.000257" iyz="1.6e-05" ixz="-0.0"/>
+  </inertial>
+  <visual>
+    <origin xyz="0.42733 -0.410572 0.281864" rpy="0 0 0"/>
     <geometry>
       <mesh filename="package://Assemblage_description/meshes/wheel3_1.stl" scale="0.001 0.001 0.001"/>
@@ -118,5 +141,5 @@
   </visual>
   <collision>
-    <origin xyz="0.408112 -0.493016 0.417916" rpy="0 0 0"/>
+    <origin xyz="0.42733 -0.410572 0.281864" rpy="0 0 0"/>
     <geometry>
       <mesh filename="package://Assemblage_description/meshes/wheel3_1.stl" scale="0.001 0.001 0.001"/>
@@ -126,10 +149,10 @@
 <link name="wheel4_1">
   <inertial>
-    <origin xyz="0.0003405329776948185 -0.010197254794899857 3.712233269614895e-06" rpy="0 0 0"/>
+    <origin xyz="0.0003392711202230836 -0.010196510227618527 -1.9767207815879484e-05" rpy="0 0 0"/>
     <mass value="1.592763813314383"/>
-    <inertia ixx="0.010896" iyy="0.018605" izz="0.010887" ixy="-0.000257" iyz="-2e-06" ixz="0.0"/>
-  </inertial>
-  <visual>
-    <origin xyz="-0.425011 -0.493016 0.410938" rpy="0 0 0"/>
+    <inertia ixx="0.010896" iyy="0.018605" izz="0.010887" ixy="-0.000257" iyz="1.6e-05" ixz="-0.0"/>
+  </inertial>
+  <visual>
+    <origin xyz="-0.404251 -0.410572 0.333019" rpy="0 0 0"/>
     <geometry>
       <mesh filename="package://Assemblage_description/meshes/wheel4_1.stl" scale="0.001 0.001 0.001"/>
@@ -138,5 +161,5 @@
   </visual>
   <collision>
-    <origin xyz="-0.425011 -0.493016 0.410938" rpy="0 0 0"/>
+    <origin xyz="-0.404251 -0.410572 0.333019" rpy="0 0 0"/>
     <geometry>
       <mesh filename="package://Assemblage_description/meshes/wheel4_1.stl" scale="0.001 0.001 0.001"/>
@@ -146,10 +169,10 @@
 <link name="wheel2_1">
   <inertial>
-    <origin xyz="-0.0003401832155410234 0.010196488127690917 3.712233260733111e-06" rpy="0 0 0"/>
+    <origin xyz="-0.0003399213580693172 0.010197232694972913 -1.9767207816323573e-05" rpy="0 0 0"/>
     <mass value="1.592763813314383"/>
-    <inertia ixx="0.010896" iyy="0.018605" izz="0.010887" ixy="-0.000257" iyz="2e-06" ixz="-0.0"/>
-  </inertial>
-  <visual>
-    <origin xyz="0.411798 0.289181 0.410938" rpy="0 0 0"/>
+    <inertia ixx="0.010896" iyy="0.018605" izz="0.010887" ixy="-0.000257" iyz="-1.6e-05" ixz="0.0"/>
+  </inertial>
+  <visual>
+    <origin xyz="0.391037 0.370625 0.333019" rpy="0 0 0"/>
     <geometry>
       <mesh filename="package://Assemblage_description/meshes/wheel2_1.stl" scale="0.001 0.001 0.001"/>
@@ -158,5 +181,5 @@
   </visual>
   <collision>
-    <origin xyz="0.411798 0.289181 0.410938" rpy="0 0 0"/>
+    <origin xyz="0.391037 0.370625 0.333019" rpy="0 0 0"/>
     <geometry>
       <mesh filename="package://Assemblage_description/meshes/wheel2_1.stl" scale="0.001 0.001 0.001"/>
@@ -166,10 +189,10 @@
 <link name="wheel1_1">
   <inertial>
-    <origin xyz="-0.0003397209476816987 0.010196488127692138 3.6630334383502827e-06" rpy="0 0 0"/>
+    <origin xyz="-0.0003391418658636458 0.010197232694973468 -2.0063309200568646e-05" rpy="0 0 0"/>
     <mass value="1.592763813314383"/>
-    <inertia ixx="0.010896" iyy="0.018605" izz="0.010887" ixy="-0.000257" iyz="2e-06" ixz="-0.0"/>
-  </inertial>
-  <visual>
-    <origin xyz="-0.421325 0.289181 0.417916" rpy="0 0 0"/>
+    <inertia ixx="0.010896" iyy="0.018605" izz="0.010887" ixy="-0.000257" iyz="-1.6e-05" ixz="0.0"/>
+  </inertial>
+  <visual>
+    <origin xyz="-0.440543 0.370625 0.281864" rpy="0 0 0"/>
     <geometry>
       <mesh filename="package://Assemblage_description/meshes/wheel1_1.stl" scale="0.001 0.001 0.001"/>
@@ -178,5 +201,5 @@
   </visual>
   <collision>
-    <origin xyz="-0.421325 0.289181 0.417916" rpy="0 0 0"/>
+    <origin xyz="-0.440543 0.370625 0.281864" rpy="0 0 0"/>
     <geometry>
       <mesh filename="package://Assemblage_description/meshes/wheel1_1.stl" scale="0.001 0.001 0.001"/>
@@ -186,10 +209,10 @@
 <link name="hd_link2_1">
   <inertial>
-    <origin xyz="0.0033070766839577714 0.06083906580288365 0.1440505220890836" rpy="0 0 0"/>
+    <origin xyz="0.007428383283974271 0.060838810370171845 0.14389716626077925" rpy="0 0 0"/>
     <mass value="2.4452075265656514"/>
-    <inertia ixx="0.038706" iyy="0.03827" izz="0.003043" ixy="3.2e-05" iyz="0.001609" ixz="-5e-05"/>
-  </inertial>
-  <visual>
-    <origin xyz="0.228643 -0.044217 -0.046218" rpy="0 0 0"/>
+    <inertia ixx="0.038674" iyy="0.03827" izz="0.003075" ixy="7.8e-05" iyz="0.001607" ixz="-0.00107"/>
+  </inertial>
+  <visual>
+    <origin xyz="0.228643 0.037726 -0.152484" rpy="0 0 0"/>
     <geometry>
       <mesh filename="package://Assemblage_description/meshes/hd_link2_1.stl" scale="0.001 0.001 0.001"/>
@@ -198,5 +221,5 @@
   </visual>
   <collision>
-    <origin xyz="0.228643 -0.044217 -0.046218" rpy="0 0 0"/>
+    <origin xyz="0.228643 0.037726 -0.152484" rpy="0 0 0"/>
     <geometry>
       <mesh filename="package://Assemblage_description/meshes/hd_link2_1.stl" scale="0.001 0.001 0.001"/>
@@ -206,10 +229,10 @@
 <link name="hd_link3_1">
   <inertial>
-    <origin xyz="-0.18542255123016124 -0.02818843505267088 0.033215191672649136" rpy="0 0 0"/>
+    <origin xyz="-0.18506431602380205 -0.028188690485378982 0.03515465538516083" rpy="0 0 0"/>
     <mass value="0.3993227194340243"/>
-    <inertia ixx="0.000838" iyy="0.00625" izz="0.006374" ixy="4.5e-05" iyz="-5e-06" ixz="0.00018"/>
-  </inertial>
-  <visual>
-    <origin xyz="0.22795 -0.132217 -0.446313" rpy="0 0 0"/>
+    <inertia ixx="0.000842" iyy="0.00625" izz="0.00637" ixy="4.5e-05" iyz="-5e-06" ixz="0.000238"/>
+  </inertial>
+  <visual>
+    <origin xyz="0.2165 -0.050274 -0.552396" rpy="0 0 0"/>
     <geometry>
       <mesh filename="package://Assemblage_description/meshes/hd_link3_1.stl" scale="0.001 0.001 0.001"/>
@@ -218,5 +241,5 @@
   </visual>
   <collision>
-    <origin xyz="0.22795 -0.132217 -0.446313" rpy="0 0 0"/>
+    <origin xyz="0.2165 -0.050274 -0.552396" rpy="0 0 0"/>
     <geometry>
       <mesh filename="package://Assemblage_description/meshes/hd_link3_1.stl" scale="0.001 0.001 0.001"/>
@@ -226,10 +249,10 @@
 <link name="hd_link4_1">
   <inertial>
-    <origin xyz="-0.026508760059289482 0.0028968395456604734 -0.000598737646716252" rpy="0 0 0"/>
+    <origin xyz="-0.02651321084424607 0.002896584112952065 -0.0003217450612928996" rpy="0 0 0"/>
     <mass value="0.16590781468918114"/>
-    <inertia ixx="0.000197" iyy="0.000349" izz="0.000476" ixy="3.9e-05" iyz="5e-06" ixz="1e-06"/>
-  </inertial>
-  <visual>
-    <origin xyz="0.54334 -0.102573 -0.481152" rpy="0 0 0"/>
+    <inertia ixx="0.000197" iyy="0.000349" izz="0.000476" ixy="3.9e-05" iyz="5e-06" ixz="4e-06"/>
+  </inertial>
+  <visual>
+    <origin xyz="0.531508 -0.02063 -0.590536" rpy="0 0 0"/>
     <geometry>
       <mesh filename="package://Assemblage_description/meshes/hd_link4_1.stl" scale="0.001 0.001 0.001"/>
@@ -238,5 +261,5 @@
   </visual>
   <collision>
-    <origin xyz="0.54334 -0.102573 -0.481152" rpy="0 0 0"/>
+    <origin xyz="0.531508 -0.02063 -0.590536" rpy="0 0 0"/>
     <geometry>
       <mesh filename="package://Assemblage_description/meshes/hd_link4_1.stl" scale="0.001 0.001 0.001"/>
@@ -246,10 +269,10 @@
 <link name="hd_link5_1">
   <inertial>
-    <origin xyz="-0.00326876427210665 0.038460537452552596 -0.0001281048652070904" rpy="0 0 0"/>
-    <mass value="0.06877842327462741"/>
-    <inertia ixx="4.9e-05" iyy="2.9e-05" izz="4.3e-05" ixy="1e-06" iyz="0.0" ixz="0.0"/>
-  </inertial>
-  <visual>
-    <origin xyz="0.63704 -0.060573 -0.481315" rpy="0 0 0"/>
+    <origin xyz="-0.0032697164246294763 0.03846028201984416 -9.33050693235904e-05" rpy="0 0 0"/>
+    <mass value="0.06877842327462745"/>
+    <inertia ixx="4.9e-05" iyy="2.9e-05" izz="4.3e-05" ixy="1e-06" iyz="0.0" ixz="-0.0"/>
+  </inertial>
+  <visual>
+    <origin xyz="0.625201 0.02137 -0.591679" rpy="0 0 0"/>
     <geometry>
       <mesh filename="package://Assemblage_description/meshes/hd_link5_1.stl" scale="0.001 0.001 0.001"/>
@@ -258,5 +281,5 @@
   </visual>
   <collision>
-    <origin xyz="0.63704 -0.060573 -0.481315" rpy="0 0 0"/>
+    <origin xyz="0.625201 0.02137 -0.591679" rpy="0 0 0"/>
     <geometry>
       <mesh filename="package://Assemblage_description/meshes/hd_link5_1.stl" scale="0.001 0.001 0.001"/>
@@ -266,10 +289,10 @@
 <link name="hd_link6_1">
   <inertial>
-    <origin xyz="-0.03520188089997378 -0.0007184800362615151 0.000553267969914728" rpy="0 0 0"/>
+    <origin xyz="-0.03519419436746607 -0.0007187354689699374 0.0009221743273718497" rpy="0 0 0"/>
     <mass value="0.11153016933793788"/>
-    <inertia ixx="0.000117" iyy="0.000166" izz="0.000263" ixy="-2e-06" iyz="-1e-06" ixz="-1e-06"/>
-  </inertial>
-  <visual>
-    <origin xyz="0.66404 -0.102533 -0.48115" rpy="0 0 0"/>
+    <inertia ixx="0.000117" iyy="0.000166" izz="0.000263" ixy="-2e-06" iyz="-1e-06" ixz="1e-06"/>
+  </inertial>
+  <visual>
+    <origin xyz="0.652201 -0.02059 -0.591797" rpy="0 0 0"/>
     <geometry>
       <mesh filename="package://Assemblage_description/meshes/hd_link6_1.stl" scale="0.001 0.001 0.001"/>
@@ -278,5 +301,5 @@
   </visual>
   <collision>
-    <origin xyz="0.66404 -0.102533 -0.48115" rpy="0 0 0"/>
+    <origin xyz="0.652201 -0.02059 -0.591797" rpy="0 0 0"/>
     <geometry>
       <mesh filename="package://Assemblage_description/meshes/hd_link6_1.stl" scale="0.001 0.001 0.001"/>
@@ -286,10 +309,10 @@
 <link name="hd_finger2_1">
   <inertial>
-    <origin xyz="0.36572155404860496 -0.7471770274512002 -0.09385171158022082" rpy="0 0 0"/>
+    <origin xyz="0.47666706754454413 -0.7361417133269437 -0.01622358994727202" rpy="0 0 0"/>
     <mass value="0.025342855198124774"/>
     <inertia ixx="4e-06" iyy="1.8e-05" izz="1.6e-05" ixy="-2e-06" iyz="-0.0" ixz="-2e-06"/>
   </inertial>
   <visual>
-    <origin xyz="1.132411 -0.857299 -0.577422" rpy="0 0 0"/>
+    <origin xyz="1.231487 -0.764267 -0.611515" rpy="0 0 0"/>
     <geometry>
       <mesh filename="package://Assemblage_description/meshes/hd_finger2_1.stl" scale="0.001 0.001 0.001"/>
@@ -298,5 +321,5 @@
   </visual>
   <collision>
-    <origin xyz="1.132411 -0.857299 -0.577422" rpy="0 0 0"/>
+    <origin xyz="1.231487 -0.764267 -0.611515" rpy="0 0 0"/>
     <geometry>
       <mesh filename="package://Assemblage_description/meshes/hd_finger2_1.stl" scale="0.001 0.001 0.001"/>
@@ -306,10 +329,10 @@
 <link name="hd_finger1_1">
   <inertial>
-    <origin xyz="0.34237822893598846 -0.7617001148724551 -0.1442671674369853" rpy="0 0 0"/>
+    <origin xyz="0.4527983426832546 -0.7504874421753438 -0.06638458975098571" rpy="0 0 0"/>
     <mass value="0.025342855198124774"/>
     <inertia ixx="4e-06" iyy="1.8e-05" izz="1.6e-05" ixy="2e-06" iyz="-0.0" ixz="2e-06"/>
   </inertial>
   <visual>
-    <origin xyz="1.10949 -0.856977 -0.62175" rpy="0 0 0"/>
+    <origin xyz="1.208101 -0.764188 -0.655601" rpy="0 0 0"/>
     <geometry>
       <mesh filename="package://Assemblage_description/meshes/hd_finger1_1.stl" scale="0.001 0.001 0.001"/>
@@ -318,5 +341,5 @@
   </visual>
   <collision>
-    <origin xyz="1.10949 -0.856977 -0.62175" rpy="0 0 0"/>
+    <origin xyz="1.208101 -0.764188 -0.655601" rpy="0 0 0"/>
     <geometry>
       <mesh filename="package://Assemblage_description/meshes/hd_finger1_1.stl" scale="0.001 0.001 0.001"/>
@@ -326,10 +349,10 @@
 <link name="hd_motor_j3_1">
   <inertial>
-    <origin xyz="-0.26883632684956255 0.15032394640210167 0.12504846034721717" rpy="0 0 0"/>
+    <origin xyz="-0.3146867524268133 0.14188869096939155 0.25591208107402835" rpy="0 0 0"/>
     <mass value="0.11925838600046076"/>
-    <inertia ixx="0.000514" iyy="0.000525" izz="2.4e-05" ixy="-0.0" iyz="-0.0" ixz="-7.3e-05"/>
-  </inertial>
-  <visual>
-    <origin xyz="-0.12039 0.049107 -0.176255" rpy="0 0 0"/>
+    <inertia ixx="0.00051" iyy="0.000525" izz="2.9e-05" ixy="-0.0" iyz="-0.0" ixz="-8.7e-05"/>
+  </inertial>
+  <visual>
+    <origin xyz="-0.173508 0.122615 -0.149258" rpy="0 0 0"/>
     <geometry>
       <mesh filename="package://Assemblage_description/meshes/hd_motor_j3_1.stl" scale="0.001 0.001 0.001"/>
@@ -338,5 +361,5 @@
   </visual>
   <collision>
-    <origin xyz="-0.12039 0.049107 -0.176255" rpy="0 0 0"/>
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