Commit message: new compiled onyx urdf

File: kinematics/rover_description/description/onyx_compiled.urdf (robot description, URDF)
Before this commit: robot new_hd, 11 links, 11 joints
Links:
- added link base_link
- added link caster_axis, mass 0.25; collision cylinder length=0.41 radius=0.005; visual cylinder length=0.41 radius=0.005
- added link caster_wheel, mass 15; collision cylinder length=0.05 radius=0.05; visual cylinder length=0.05 radius=0.05
- added link chassis_link, mass 50; visual mesh filename=package://rover_description/meshes/base_link.stl scale=0.001 0.001 0.001
- added link left_leg, mass 1.6615144825592312; collision mesh filename=package://rover_description/meshes/pivot_gauche_1.stl scale=0.001 0.001 0.001; visual mesh filename=package://rover_description/meshes/pivot_gauche_1.stl scale=0.001 0.001 0.001
- added link lidar_axis, mass 0.25; collision cylinder length=0.24 radius=0.005; visual cylinder length=0.24 radius=0.005
- added link right_leg, mass 1.6615144825592312; collision mesh filename=package://rover_description/meshes/pivot_droit_1.stl scale=0.001 0.001 0.001; visual mesh filename=package://rover_description/meshes/pivot_droit_1.stl scale=0.001 0.001 0.001
- added link steering1_link, mass 0.3543584805415501; collision mesh filename=package://rover_description/meshes/steering_3.stl scale=0.001 0.001 0.001; visual mesh filename=package://rover_description/meshes/steering_3.stl scale=0.001 0.001 0.001
- added link steering2_link, mass 0.3543584805415501; collision mesh filename=package://rover_description/meshes/steering_4.stl scale=0.001 0.001 0.001; visual mesh filename=package://rover_description/meshes/steering_4.stl scale=0.001 0.001 0.001
- added link steering3_link, mass 0.3543584805415501; collision mesh filename=package://rover_description/meshes/steering_1.stl scale=0.001 0.001 0.001; visual mesh filename=package://rover_description/meshes/steering_1.stl scale=0.001 0.001 0.001
- added link steering4_link, mass 0.3543584805415501; collision mesh filename=package://rover_description/meshes/steering_2.stl scale=0.001 0.001 0.001; visual mesh filename=package://rover_description/meshes/steering_2.stl scale=0.001 0.001 0.001
- added link wheel1_1ink, mass 1.592763813314383; collision mesh filename=package://rover_description/meshes/wheel2_1.stl scale=0.001 0.001 0.001; visual mesh filename=package://rover_description/meshes/wheel2_1.stl scale=0.001 0.001 0.001
- added link wheel2_1ink, mass 1.592763813314383; collision mesh filename=package://rover_description/meshes/wheel3_1.stl scale=0.001 0.001 0.001; visual mesh filename=package://rover_description/meshes/wheel3_1.stl scale=0.001 0.001 0.001
- added link wheel3_1ink, mass 1.592763813314383; collision mesh filename=package://rover_description/meshes/wheel4_1.stl scale=0.001 0.001 0.001; visual mesh filename=package://rover_description/meshes/wheel4_1.stl scale=0.001 0.001 0.001
- added link wheel4_1ink, mass 1.592763813314383; collision mesh filename=package://rover_description/meshes/wheel1_1.stl scale=0.001 0.001 0.001; visual mesh filename=package://rover_description/meshes/wheel1_1.stl scale=0.001 0.001 0.001
Joints:
- added joint caster_axis_to_caster_wheel: type continuous, parent caster_axis, child caster_wheel, origin xyz=0 0 -0.25 rpy=1.5707963267948966 0 0, axis 0 0 1
- added joint chassis_joint: type fixed, parent base_link, child chassis_link, origin xyz=0 0 0  rpy=0 0 0, axis 0.0 1.0 0.0
- added joint chassis_to_caster_axis: type continuous, parent chassis_link, child caster_axis, origin xyz=0.3 0.0 -0.225 rpy=0 -0.6 0, axis 0 0 1
- added joint chassis_to_lidar_axis: type fixed, parent chassis_link, child lidar_axis, origin xyz=0.2 0.20 0.12 rpy=0 0 0
- added joint driving1: type fixed, parent steering1_link, child wheel1_1ink, origin xyz=0.017134 -0.016691 -0.269457 rpy=0 0 0, axis 0.033267 -0.999444 0.002046
- added joint driving2: type fixed, parent steering2_link, child wheel2_1ink, origin xyz=-0.017133 0.01669 -0.269456 rpy=0 0 0, axis -0.033267 0.999444 0.002046
- added joint driving3: type fixed, parent steering3_link, child wheel3_1ink, origin xyz=-0.017133 0.01669 -0.269457 rpy=0 0 0, axis -0.033267 0.999444 0.002046
- added joint driving4: type fixed, parent steering4_link, child wheel4_1ink, origin xyz=0.017133 -0.016691 -0.269456 rpy=0 0 0, axis 0.033267 -0.999444 0.002046
- added joint left_pivot: type fixed, parent chassis_link, child left_leg, origin xyz=0 -0.210526 -0.021516 rpy=0 0 0, axis 0.0 1.0 0.0, mimic joint=right_pivot multiplier=-1.0
- added joint right_pivot: type fixed, parent chassis_link, child right_leg, origin xyz=0 0.250474 -0.021516 rpy=0 0 0, axis 0.0 1.0 0.0
- added joint steering1: type fixed, parent left_leg, child steering1_link, origin xyz=-0.414778 -0.143408 -0.042046 rpy=0 0 0, axis 0.061399 -0.0 -0.998113
- added joint steering2: type fixed, parent right_leg, child steering2_link, origin xyz=-0.416804 0.143408 0.009108 rpy=0 0 0, axis 0.061399 -0.0 0.998113
- added joint steering3: type fixed, parent right_leg, child steering3_link, origin xyz=0.414777 0.143408 -0.042046 rpy=0 0 0, axis -0.061399 0.0 -0.998113
- added joint steering4: type fixed, parent left_leg, child steering4_link, origin xyz=0.416803 -0.143408 0.009108 rpy=0 0 0, axis -0.061399 0.0 0.998113
