Commit message: moveit servo kinda integrated not working

File: kinematics/kerby_description/urdf/kerby_truncated.urdf.xacro (robot description, xacro)
@@ -187,4 +187,19 @@
   </collision>
 </link>
+<!-- <link name="fake_gripper">
+  <visual>
+    <origin xyz="0.652201 -0.02059 -0.591797" rpy="0 0 0"/>
+    <geometry>
+      <mesh filename="package://kerby_description/meshes/hd_link6_1.stl" scale="0.001 0.001 0.001"/>
+    </geometry>
+    <material name="silver"/>
+  </visual>
+  <collision>
+    <origin xyz="0.652201 -0.02059 -0.591797" rpy="0 0 0"/>
+    <geometry>
+      <mesh filename="package://kerby_description/meshes/hd_link6_1.stl" scale="0.001 0.001 0.001"/>
+    </geometry>
+  </collision>
+</link> -->
 <joint name="joint2" type="revolute">
   <origin xyz="0.0 -0.0577 0.117" rpy="0 0 0"/>

Commit message: mobeit servooo

File: kinematics/kerby_description/urdf/kerby_truncated.urdf.xacro (robot description, xacro)
@@ -5,5 +5,5 @@
 <xacro:include filename="$(find kerby_description)/urdf/kerby.gazebo" />
 <xacro:property name="rpm_to_Radps" value="${2*pi/60.0}" />     <!-- rotations per minute to Rad per second conversion -->
-<xacro:property name="velocity_scaling" value="10.0" />     <!-- allows to scale all max velocities down at once -->
+<xacro:property name="velocity_scaling" value="2.0" />     <!-- allows to scale all max velocities down at once -->
 <xacro:macro name="aaa_joint_limits" params="lower:=0.0 upper:=0.0 velocity:=${rpm_to_Radps} effort:=100.0">
   <limit lower="${lower}" upper="${upper}" velocity="${velocity}" effort="${effort}"/>
@@ -187,19 +187,19 @@
   </collision>
 </link>
-<!-- <link name="fake_gripper">
-  <visual>
+<link name="fake_gripper">
+  <!-- <visual>
+    <origin xyz="0 0 0" rpy="0 0 0"/>
+    <geometry>
+      <mesh filename="package://kerby_description/meshes/hd_link6_1.stl" scale="0.001 0.001 0.001"/>
+    </geometry>
+    <material name="silver"/>
+  </visual>
+  <collision>
     <origin xyz="0.652201 -0.02059 -0.591797" rpy="0 0 0"/>
     <geometry>
       <mesh filename="package://kerby_description/meshes/hd_link6_1.stl" scale="0.001 0.001 0.001"/>
     </geometry>
-    <material name="silver"/>
-  </visual>
-  <collision>
-    <origin xyz="0.652201 -0.02059 -0.591797" rpy="0 0 0"/>
-    <geometry>
-      <mesh filename="package://kerby_description/meshes/hd_link6_1.stl" scale="0.001 0.001 0.001"/>
-    </geometry>
-  </collision>
-</link> -->
+  </collision> -->
+</link>
 <joint name="joint2" type="revolute">
   <origin xyz="0.0 -0.0577 0.117" rpy="0 0 0"/>
@@ -249,3 +249,8 @@
   <xacro:insert_block name="joint1_limits" />
 </joint>
+<joint name="fake_gripper_joint" type="fixed">
+  <origin xyz="-0.12 0 0" rpy="0 0 0"/>
+  <parent link="hd_link6_1"/>
+  <child link="fake_gripper"/>
+</joint>
 </robot>

Commit message: still no nice frame

File: kinematics/kerby_description/urdf/kerby_truncated.urdf.xacro (robot description, xacro)
@@ -253,4 +253,5 @@
   <parent link="hd_link6_1"/>
   <child link="fake_gripper"/>
+  <!-- <limit lower="0" upper="0" velocity="0" effort="0"/> -->
 </joint>
 </robot>
