Commit message: attempt at correcting urdf zeros manually with math (my math is wrong)

File: kinematics/onyx_description/description/URDF3.urdf.xacro (robot description, xacro)
@@ -240,5 +240,5 @@
 <joint name="hd_joint1" type="continuous">
   <!-- <origin xyz="0.007012 0.143312 0.484988" rpy="0 0 0"/> -->
-  <origin xyz="0 0 0" rpy="${pi/2} 0 0"/>
+  <origin xyz="0 0 0" rpy="${pi/2} 0 -1.091427"/>
   <parent link="base"/>
   <child link="hd_link1"/>
@@ -246,9 +246,10 @@
 </joint>
 <joint name="hd_joint2" type="continuous">
-  <origin xyz="0.104169 0.1185 0.056489" rpy="0 0 0"/>
+  <origin xyz="0.104169 0.1185 0.056489" rpy="-0.4079707 0.1795091 -0.8207109"/>
   <parent link="hd_link1"/>
   <child link="hd_link2"/>
   <axis xyz="0.879067 0.0 0.476699"/>
 </joint>
+<!-- [ x: -0.8207109, y: 0.1795091, z: -0.4079707 ] -->
 <joint name="hd_joint3" type="continuous">
   <origin xyz="-0.14594 0.209699 0.269123" rpy="0 0 0"/>
@@ -298,4 +299,4 @@
   <child link="Gripper_Finger_v1__1__1"/>
   <axis xyz="0.9845 -0.100287 0.14388"/>
-</joint> -->
+</joint>
 </robot>

Commit message: urdf back to normal (with only joint 1 zero adjusted)

File: kinematics/onyx_description/description/URDF3.urdf.xacro (robot description, xacro)
@@ -246,5 +246,5 @@
 </joint>
 <joint name="hd_joint2" type="continuous">
-  <origin xyz="0.104169 0.1185 0.056489" rpy="-0.4079707 0.1795091 -0.8207109"/>
+  <origin xyz="0.104169 0.1185 0.056489" rpy="0 0 0"/>
   <parent link="hd_link1"/>
   <child link="hd_link2"/>

Commit message: moveit servo POC with onyx arm

File: kinematics/onyx_description/description/URDF3.urdf.xacro (robot description, xacro)
@@ -1,8 +1,8 @@
 <?xml version="1.0" ?>
 <robot name="new_hd" xmlns:xacro="http://www.ros.org/wiki/xacro">
-<!-- <xacro:include filename="$(find rover_description)/description/materials3.xacro" /> -->
-<!-- <xacro:include filename="$(find rover_description)/description/URDF3.trans" /> -->
-<xacro:include filename="$(find rover_description)/description/URDF3.gazebo" />
-<!-- <xacro:include filename="$(find rover_description)/description/ros2_control_arm.xacro" /> -->
+<!-- <xacro:include filename="$(find onyx_description)/description/materials3.xacro" /> -->
+<!-- <xacro:include filename="$(find onyx_description)/description/URDF3.trans" /> -->
+<xacro:include filename="$(find onyx_description)/description/URDF3.gazebo" />
+<!-- <xacro:include filename="$(find onyx_description)/description/ros2_control_arm.xacro" /> -->
 <!-- <link name="base_link"/> -->
 <joint name="hd_joint0" type="fixed">
@@ -27,5 +27,5 @@
     <origin xyz="0 0.47 -0.12" rpy="${pi/2} 0 0"/>
     <geometry>
-      <mesh filename="package://rover_description/meshes/new_hd/base_link.stl" scale="0.001 0.001 0.001"/>
+      <mesh filename="package://onyx_description/meshes/new_hd/base_link.stl" scale="0.001 0.001 0.001"/>
     </geometry>
     <material name="silver"/>
@@ -34,5 +34,5 @@
     <origin xyz="0 0.47 -0.12" rpy="${pi/2} 0 0"/>
     <geometry>
-      <mesh filename="package://rover_description/meshes/new_hd/base_link.stl" scale="0.001 0.001 0.001"/>
+      <mesh filename="package://onyx_description/meshes/new_hd/base_link.stl" scale="0.001 0.001 0.001"/>
     </geometry>
   </collision>
@@ -47,5 +47,5 @@
     <origin xyz="-0.007012 -0.143312 -0.484988" rpy="0 0 0"/>
     <geometry>
-      <mesh filename="package://rover_description/meshes/new_hd/link_1_1.stl" scale="0.001 0.001 0.001"/>
+      <mesh filename="package://onyx_description/meshes/new_hd/link_1_1.stl" scale="0.001 0.001 0.001"/>
     </geometry>
     <material name="silver"/>
@@ -54,5 +54,5 @@
     <origin xyz="-0.007012 -0.143312 -0.484988" rpy="0 0 0"/>
     <geometry>
-      <mesh filename="package://rover_description/meshes/new_hd/link_1_1.stl" scale="0.001 0.001 0.001"/>
+      <mesh filename="package://onyx_description/meshes/new_hd/link_1_1.stl" scale="0.001 0.001 0.001"/>
     </geometry>
   </collision>
@@ -67,5 +67,5 @@
     <origin xyz="-0.111181 -0.261812 -0.541477" rpy="0 0 0"/>
     <geometry>
-      <mesh filename="package://rover_description/meshes/new_hd/link_2_1.stl" scale="0.001 0.001 0.001"/>
+      <mesh filename="package://onyx_description/meshes/new_hd/link_2_1.stl" scale="0.001 0.001 0.001"/>
     </geometry>
     <material name="silver"/>
@@ -74,5 +74,5 @@
     <origin xyz="-0.111181 -0.261812 -0.541477" rpy="0 0 0"/>
     <geometry>
-      <mesh filename="package://rover_description/meshes/new_hd/link_2_1.stl" scale="0.001 0.001 0.001"/>
+      <mesh filename="package://onyx_description/meshes/new_hd/link_2_1.stl" scale="0.001 0.001 0.001"/>
     </geometry>
   </collision>
@@ -87,5 +87,5 @@
     <origin xyz="0.034759 -0.471511 -0.8106" rpy="0 0 0"/>
     <geometry>
-      <mesh filename="package://rover_description/meshes/new_hd/link_3_1.stl" scale="0.001 0.001 0.001"/>
+      <mesh filename="package://onyx_description/meshes/new_hd/link_3_1.stl" scale="0.001 0.001 0.001"/>
     </geometry>
     <material name="silver"/>
@@ -94,5 +94,5 @@
     <origin xyz="0.034759 -0.471511 -0.8106" rpy="0 0 0"/>
     <geometry>
-      <mesh filename="package://rover_description/meshes/new_hd/link_3_1.stl" scale="0.001 0.001 0.001"/>
+      <mesh filename="package://onyx_description/meshes/new_hd/link_3_1.stl" scale="0.001 0.001 0.001"/>
     </geometry>
   </collision>
@@ -107,5 +107,5 @@
     <origin xyz="0.082848 -0.485732 -0.650695" rpy="0 0 0"/>
     <geometry>
-      <mesh filename="package://rover_description/meshes/new_hd/link_4_1.stl" scale="0.001 0.001 0.001"/>
+      <mesh filename="package://onyx_description/meshes/new_hd/link_4_1.stl" scale="0.001 0.001 0.001"/>
     </geometry>
     <material name="silver"/>
@@ -114,5 +114,5 @@
     <origin xyz="0.082848 -0.485732 -0.650695" rpy="0 0 0"/>
     <geometry>
-      <mesh filename="package://rover_description/meshes/new_hd/link_4_1.stl" scale="0.001 0.001 0.001"/>
+      <mesh filename="package://onyx_description/meshes/new_hd/link_4_1.stl" scale="0.001 0.001 0.001"/>
     </geometry>
   </collision>
@@ -127,5 +127,5 @@
     <origin xyz="-0.030684 -0.519236 -0.405724" rpy="0 0 0"/>
     <geometry>
-      <mesh filename="package://rover_description/meshes/new_hd/link_5_1.stl" scale="0.001 0.001 0.001"/>
+      <mesh filename="package://onyx_description/meshes/new_hd/link_5_1.stl" scale="0.001 0.001 0.001"/>
     </geometry>
     <material name="silver"/>
@@ -134,5 +134,5 @@
     <origin xyz="-0.030684 -0.519236 -0.405724" rpy="0 0 0"/>
     <geometry>
-      <mesh filename="package://rover_description/meshes/new_hd/link_5_1.stl" scale="0.001 0.001 0.001"/>
+      <mesh filename="package://onyx_description/meshes/new_hd/link_5_1.stl" scale="0.001 0.001 0.001"/>
     </geometry>
   </collision>
@@ -147,5 +147,5 @@
     <origin xyz="-0.148761 -0.629862 -0.449364" rpy="0 0 0"/>
     <geometry>
-      <mesh filename="package://rover_description/meshes/new_hd/link_6_1.stl" scale="0.001 0.001 0.001"/>
+      <mesh filename="package://onyx_description/meshes/new_hd/link_6_1.stl" scale="0.001 0.001 0.001"/>
     </geometry>
     <material name="silver"/>
@@ -154,5 +154,5 @@
     <origin xyz="-0.148761 -0.629862 -0.449364" rpy="0 0 0"/>
     <geometry>
-      <mesh filename="package://rover_description/meshes/new_hd/link_6_1.stl" scale="0.001 0.001 0.001"/>
+      <mesh filename="package://onyx_description/meshes/new_hd/link_6_1.stl" scale="0.001 0.001 0.001"/>
     </geometry>
   </collision>
@@ -167,5 +167,5 @@
     <origin xyz="-0.139762 -0.725909 -0.421506" rpy="0 0 0"/>
     <geometry>
-      <mesh filename="package://rover_description/meshes/new_hd/Gripper_Arcs_v1_1.stl" scale="0.001 0.001 0.001"/>
+      <mesh filename="package://onyx_description/meshes/new_hd/Gripper_Arcs_v1_1.stl" scale="0.001 0.001 0.001"/>
     </geometry>
     <material name="silver"/>
@@ -174,5 +174,5 @@
     <origin xyz="-0.139762 -0.725909 -0.421506" rpy="0 0 0"/>
     <geometry>
-      <mesh filename="package://rover_description/meshes/new_hd/Gripper_Arcs_v1_1.stl" scale="0.001 0.001 0.001"/>
+      <mesh filename="package://onyx_description/meshes/new_hd/Gripper_Arcs_v1_1.stl" scale="0.001 0.001 0.001"/>
     </geometry>
   </collision>
@@ -187,5 +187,5 @@
     <origin xyz="-0.153478 -0.800615 -0.379727" rpy="0 0 0"/>
     <geometry>
-      <mesh filename="package://rover_description/meshes/new_hd/Gripper_Finger_v1_1.stl" scale="0.001 0.001 0.001"/>
+      <mesh filename="package://onyx_description/meshes/new_hd/Gripper_Finger_v1_1.stl" scale="0.001 0.001 0.001"/>
     </geometry>
     <material name="silver"/>
@@ -194,5 +194,5 @@
     <origin xyz="-0.153478 -0.800615 -0.379727" rpy="0 0 0"/>
     <geometry>
-      <mesh filename="package://rover_description/meshes/new_hd/Gripper_Finger_v1_1.stl" scale="0.001 0.001 0.001"/>
+      <mesh filename="package://onyx_description/meshes/new_hd/Gripper_Finger_v1_1.stl" scale="0.001 0.001 0.001"/>
     </geometry>
   </collision>
@@ -207,5 +207,5 @@
     <origin xyz="-0.135804 -0.729418 -0.451036" rpy="0 0 0"/>
     <geometry>
-      <mesh filename="package://rover_description/meshes/new_hd/Gripper_Arcs_v1__2__1.stl" scale="0.001 0.001 0.001"/>
+      <mesh filename="package://onyx_description/meshes/new_hd/Gripper_Arcs_v1__2__1.stl" scale="0.001 0.001 0.001"/>
     </geometry>
     <material name="silver"/>
@@ -214,5 +214,5 @@
     <origin xyz="-0.135804 -0.729418 -0.451036" rpy="0 0 0"/>
     <geometry>
-      <mesh filename="package://rover_description/meshes/new_hd/Gripper_Arcs_v1__2__1.stl" scale="0.001 0.001 0.001"/>
+      <mesh filename="package://onyx_description/meshes/new_hd/Gripper_Arcs_v1__2__1.stl" scale="0.001 0.001 0.001"/>
     </geometry>
   </collision>
@@ -227,5 +227,5 @@
     <origin xyz="-0.142591 -0.81484 -0.464138" rpy="0 0 0"/>
     <geometry>
-      <mesh filename="package://rover_description/meshes/new_hd/Gripper_Finger_v1__1__1.stl" scale="0.001 0.001 0.001"/>
+      <mesh filename="package://onyx_description/meshes/new_hd/Gripper_Finger_v1__1__1.stl" scale="0.001 0.001 0.001"/>
     </geometry>
     <material name="silver"/>
@@ -234,5 +234,5 @@
     <origin xyz="-0.142591 -0.81484 -0.464138" rpy="0 0 0"/>
     <geometry>
-      <mesh filename="package://rover_description/meshes/new_hd/Gripper_Finger_v1__1__1.stl" scale="0.001 0.001 0.001"/>
+      <mesh filename="package://onyx_description/meshes/new_hd/Gripper_Finger_v1__1__1.stl" scale="0.001 0.001 0.001"/>
     </geometry>
   </collision>

File: kinematics/onyx_description/description/onyx.urdf.xacro (robot description, xacro)
@@ -4,10 +4,10 @@
 <xacro:include filename="$(find onyx_description)/description/kerby.trans" />
 <xacro:include filename="$(find onyx_description)/description/kerby.gazebo" />
-<!-- <xacro:include filename="package://rover_description/description/ouster.xacro" />
-<xacro:include filename="package://rover_description/description/imu.xacro" />  -->
+<!-- <xacro:include filename="package://onyx_description/description/ouster.xacro" />
+<xacro:include filename="package://onyx_description/description/imu.xacro" />  -->
 <xacro:include filename="$(find onyx_description)/description/inertial_macros.xacro" />
-<!-- <xacro:include filename="package://rover_description/description/oakd_camera.xacro" /> -->
+<!-- <xacro:include filename="package://onyx_description/description/oakd_camera.xacro" /> -->
 <xacro:include filename="$(find onyx_description)/description/URDF3.urdf.xacro" />
-<!-- <xacro:include filename="package://rover_description/description/ros2_control_arm.xacro" /> -->
+<!-- <xacro:include filename="package://onyx_description/description/ros2_control_arm.xacro" /> -->
 <link name="base_link"></link>
 <joint name="chassis_joint" type="fixed">
@@ -27,5 +27,5 @@
     <origin xyz="0 0 0" rpy="0 0 0"/>
     <geometry>
-      <mesh filename="package://rover_description/meshes/base_link.stl" scale="0.001 0.001 0.001"/>
+      <mesh filename="package://onyx_description/meshes/base_link.stl" scale="0.001 0.001 0.001"/>
     </geometry>
     <material name="blue"/>
@@ -34,5 +34,5 @@
     <origin xyz="0 0 0" rpy="0 0 0"/>
     <geometry>
-      <mesh filename="package://rover_description/meshes/base_link.stl" scale="0.001 0.001 0.001"/>
+      <mesh filename="package://onyx_description/meshes/base_link.stl" scale="0.001 0.001 0.001"/>
     </geometry>
   </collision> -->
@@ -47,5 +47,5 @@
     <origin xyz="-0.421384 -0.393882 0.063562" rpy="0 0 0"/>
     <geometry>
-      <mesh filename="package://rover_description/meshes/steering_1.stl" scale="0.001 0.001 0.001"/>
+      <mesh filename="package://onyx_description/meshes/steering_1.stl" scale="0.001 0.001 0.001"/>
     </geometry>
     <material name="silver"/>
@@ -54,5 +54,5 @@
     <origin xyz="-0.421384 -0.393882 0.063562" rpy="0 0 0"/>
     <geometry>
-      <mesh filename="package://rover_description/meshes/steering_1.stl" scale="0.001 0.001 0.001"/>
+      <mesh filename="package://onyx_description/meshes/steering_1.stl" scale="0.001 0.001 0.001"/>
     </geometry>
   </collision>
@@ -67,5 +67,5 @@
     <origin xyz="-0.42341 0.353934 0.012408" rpy="0 0 0"/>
     <geometry>
-      <mesh filename="package://rover_description/meshes/steering_2.stl" scale="0.001 0.001 0.001"/>
+      <mesh filename="package://onyx_description/meshes/steering_2.stl" scale="0.001 0.001 0.001"/>
     </geometry>
     <material name="silver"/>
@@ -74,5 +74,5 @@
     <origin xyz="-0.42341 0.353934 0.012408" rpy="0 0 0"/>
     <geometry>
-      <mesh filename="package://rover_description/meshes/steering_2.stl" scale="0.001 0.001 0.001"/>
+      <mesh filename="package://onyx_description/meshes/steering_2.stl" scale="0.001 0.001 0.001"/>
     </geometry>
   </collision>
@@ -87,5 +87,5 @@
     <origin xyz="0.408171 0.353934 0.063562" rpy="0 0 0"/>
     <geometry>
-      <mesh filename="package://rover_description/meshes/steering_3.stl" scale="0.001 0.001 0.001"/>
+      <mesh filename="package://onyx_description/meshes/steering_3.stl" scale="0.001 0.001 0.001"/>
     </geometry>
     <material name="silver"/>
@@ -94,5 +94,5 @@
     <origin xyz="0.408171 0.353934 0.063562" rpy="0 0 0"/>
     <geometry>
-      <mesh filename="package://rover_description/meshes/steering_3.stl" scale="0.001 0.001 0.001"/>
+      <mesh filename="package://onyx_description/meshes/steering_3.stl" scale="0.001 0.001 0.001"/>
     </geometry>
   </collision>
@@ -107,5 +107,5 @@
     <origin xyz="0.410197 -0.393882 0.012408" rpy="0 0 0"/>
     <geometry>
-      <mesh filename="package://rover_description/meshes/steering_4.stl" scale="0.001 0.001 0.001"/>
+      <mesh filename="package://onyx_description/meshes/steering_4.stl" scale="0.001 0.001 0.001"/>
     </geometry>
     <material name="silver"/>
@@ -114,5 +114,5 @@
     <origin xyz="0.410197 -0.393882 0.012408" rpy="0 0 0"/>
     <geometry>
-      <mesh filename="package://rover_description/meshes/steering_4.stl" scale="0.001 0.001 0.001"/>
+      <mesh filename="package://onyx_description/meshes/steering_4.stl" scale="0.001 0.001 0.001"/>
     </geometry>
   </collision>
@@ -127,5 +127,5 @@
     <origin xyz="0.42733 -0.410572 0.281864" rpy="0 0 0"/>
     <geometry>
-      <mesh filename="package://rover_description/meshes/wheel3_1.stl" scale="0.001 0.001 0.001"/>
+      <mesh filename="package://onyx_description/meshes/wheel3_1.stl" scale="0.001 0.001 0.001"/>
     </geometry>
     <material name="pink"/>
@@ -134,5 +134,5 @@
     <origin xyz="0.42733 -0.410572 0.281864" rpy="0 0 0"/>
     <geometry>
-      <mesh filename="package://rover_description/meshes/wheel3_1.stl" scale="0.001 0.001 0.001"/>
+      <mesh filename="package://onyx_description/meshes/wheel3_1.stl" scale="0.001 0.001 0.001"/>
     </geometry>
   </collision>
@@ -147,5 +147,5 @@
     <origin xyz="-0.404251 -0.410572 0.333019" rpy="0 0 0"/>
     <geometry>
-      <mesh filename="package://rover_description/meshes/wheel4_1.stl" scale="0.001 0.001 0.001"/>
+      <mesh filename="package://onyx_description/meshes/wheel4_1.stl" scale="0.001 0.001 0.001"/>
     </geometry>
     <material name="pink"/>
@@ -154,5 +154,5 @@
     <origin xyz="-0.404251 -0.410572 0.333019" rpy="0 0 0"/>
     <geometry>
-      <mesh filename="package://rover_description/meshes/wheel4_1.stl" scale="0.001 0.001 0.001"/>
+      <mesh filename="package://onyx_description/meshes/wheel4_1.stl" scale="0.001 0.001 0.001"/>
     </geometry>
   </collision>
@@ -167,5 +167,5 @@
     <origin xyz="0.391037 0.370625 0.333019" rpy="0 0 0"/>
     <geometry>
-      <mesh filename="package://rover_description/meshes/wheel2_1.stl" scale="0.001 0.001 0.001"/>
+      <mesh filename="package://onyx_description/meshes/wheel2_1.stl" scale="0.001 0.001 0.001"/>
     </geometry>
     <material name="pink"/>
@@ -174,5 +174,5 @@
     <origin xyz="0.391037 0.370625 0.333019" rpy="0 0 0"/>
     <geometry>
-      <mesh filename="package://rover_description/meshes/wheel2_1.stl" scale="0.001 0.001 0.001"/>
+      <mesh filename="package://onyx_description/meshes/wheel2_1.stl" scale="0.001 0.001 0.001"/>
     </geometry>
   </collision>
@@ -187,5 +187,5 @@
     <origin xyz="-0.440543 0.370625 0.281864" rpy="0 0 0"/>
     <geometry>
-      <mesh filename="package://rover_description/meshes/wheel1_1.stl" scale="0.001 0.001 0.001"/>
+      <mesh filename="package://onyx_description/meshes/wheel1_1.stl" scale="0.001 0.001 0.001"/>
     </geometry>
     <material name="pink"/>
@@ -194,5 +194,5 @@
     <origin xyz="-0.440543 0.370625 0.281864" rpy="0 0 0"/>
     <geometry>
-      <mesh filename="package://rover_description/meshes/wheel1_1.stl" scale="0.001 0.001 0.001"/>
+      <mesh filename="package://onyx_description/meshes/wheel1_1.stl" scale="0.001 0.001 0.001"/>
     </geometry>
   </collision>
@@ -207,5 +207,5 @@
     <origin xyz="-0.006607 -0.250474 0.021516" rpy="0 0 0"/>
     <geometry>
-      <mesh filename="package://rover_description/meshes/pivot_droit_1.stl" scale="0.001 0.001 0.001"/>
+      <mesh filename="package://onyx_description/meshes/pivot_droit_1.stl" scale="0.001 0.001 0.001"/>
     </geometry>
     <material name="black"/>
@@ -214,5 +214,5 @@
     <origin xyz="-0.006607 -0.250474 0.021516" rpy="0 0 0"/>
     <geometry>
-      <mesh filename="package://rover_description/meshes/pivot_droit_1.stl" scale="0.001 0.001 0.001"/>
+      <mesh filename="package://onyx_description/meshes/pivot_droit_1.stl" scale="0.001 0.001 0.001"/>
     </geometry>
   </collision>
@@ -227,5 +227,5 @@
     <origin xyz="-0.006607 0.210526 0.021516" rpy="0 0 0"/>
     <geometry>
-      <mesh filename="package://rover_description/meshes/pivot_gauche_1.stl" scale="0.001 0.001 0.001"/>
+      <mesh filename="package://onyx_description/meshes/pivot_gauche_1.stl" scale="0.001 0.001 0.001"/>
     </geometry>
     <material name="black"/>
@@ -234,5 +234,5 @@
     <origin xyz="-0.006607 0.210526 0.021516" rpy="0 0 0"/>
     <geometry>
-      <mesh filename="package://rover_description/meshes/pivot_gauche_1.stl" scale="0.001 0.001 0.001"/>
+      <mesh filename="package://onyx_description/meshes/pivot_gauche_1.stl" scale="0.001 0.001 0.001"/>
     </geometry>
   </collision>

Commit message: new urdf

File: kinematics/onyx_description/description/URDF3.urdf.xacro (robot description, xacro)
@@ -5,4 +5,27 @@
 <xacro:include filename="$(find onyx_description)/description/URDF3.gazebo" />
 <!-- <xacro:include filename="$(find onyx_description)/description/ros2_control_arm.xacro" /> -->
+<xacro:property name="rpm_to_Radps" value="${2*pi/60.0}" />     <!-- rotations per minute to Rad per second conversion -->
+<xacro:property name="velocity_scaling" value="5.0" />     <!-- allows to scale all max velocities down at once -->
+<xacro:macro name="aaa_joint_limits" params="lower:=0.0 upper:=0.0 velocity:=${rpm_to_Radps} effort:=100.0">
+  <limit lower="${lower}" upper="${upper}" velocity="${velocity}" effort="${effort}"/>
+</xacro:macro>
+<xacro:property name="joint1_limits">
+  <xacro:aaa_joint_limits lower="${-10*pi}" upper="${10*pi}" velocity="${1.83 * rpm_to_Radps * velocity_scaling}" />
+</xacro:property>
+<xacro:property name="joint2_limits">
+  <xacro:aaa_joint_limits lower="${-10*pi}" upper="${10*pi}" velocity="${1.377 * rpm_to_Radps * velocity_scaling}" />
+</xacro:property>
+<xacro:property name="joint3_limits">
+  <xacro:aaa_joint_limits lower="${-10*pi}" upper="${10*pi}" velocity="${1.377 * rpm_to_Radps * velocity_scaling}" />
+</xacro:property>
+<xacro:property name="joint4_limits">
+  <xacro:aaa_joint_limits lower="${-10*pi}" upper="${10*pi}" velocity="${1.83 * rpm_to_Radps * velocity_scaling}" />
+</xacro:property>
+<xacro:property name="joint5_limits">
+  <xacro:aaa_joint_limits lower="${-10*pi}" upper="${10*pi}" velocity="${1.83 * rpm_to_Radps * velocity_scaling}" />
+</xacro:property>
+<xacro:property name="joint6_limits">
+  <xacro:aaa_joint_limits lower="${-10*pi}" upper="${10*pi}" velocity="${1.83 * rpm_to_Radps * velocity_scaling}" />
+</xacro:property>
 <!-- <link name="base_link"/> -->
 <joint name="hd_joint0" type="fixed">
@@ -238,5 +261,5 @@
   </collision>
 </link>
-<joint name="hd_joint1" type="continuous">
+<joint name="hd_joint1" type="revolute">
   <!-- <origin xyz="0.007012 0.143312 0.484988" rpy="0 0 0"/> -->
   <origin xyz="0 0 0" rpy="${pi/2} 0 -1.091427"/>
@@ -244,35 +267,41 @@
   <child link="hd_link1"/>
   <axis xyz="0 1 0"/>
-</joint>
-<joint name="hd_joint2" type="continuous">
+  <xacro:insert_block name="joint1_limits"/>
+</joint>
+<joint name="hd_joint2" type="revolute">
   <origin xyz="0.104169 0.1185 0.056489" rpy="0 0 0"/>
   <parent link="hd_link1"/>
   <child link="hd_link2"/>
   <axis xyz="0.879067 0.0 0.476699"/>
+  <xacro:insert_block name="joint2_limits"/>
 </joint>
 <!-- [ x: -0.8207109, y: 0.1795091, z: -0.4079707 ] -->
-<joint name="hd_joint3" type="continuous">
+<joint name="hd_joint3" type="revolute">
   <origin xyz="-0.14594 0.209699 0.269123" rpy="0 0 0"/>
   <parent link="hd_link2"/>
   <child link="hd_link3"/>
   <axis xyz="-0.879067 -0.0 -0.476699"/>
-</joint>
-<joint name="hd_joint4" type="continuous">
+  <xacro:insert_block name="joint3_limits"/>
+</joint>
+<joint name="hd_joint4" type="revolute">
   <origin xyz="-0.048089 0.014221 -0.159905" rpy="0 0 0"/>
   <parent link="hd_link3"/>
   <child link="hd_link4"/>
   <axis xyz="0.473254 0.120008 -0.872713"/>
-</joint>
-<joint name="hd_joint5" type="continuous">
+  <xacro:insert_block name="joint4_limits"/>
+</joint>
+<joint name="hd_joint5" type="revolute">
   <origin xyz="0.113532 0.033504 -0.244971" rpy="0 0 0"/>
   <parent link="hd_link4"/>
   <child link="hd_link5"/>
   <axis xyz="0.880882 -0.054511 0.470187"/>
-</joint>
-<joint name="hd_joint6" type="continuous">
+  <xacro:insert_block name="joint5_limits"/>
+</joint>
+<joint name="hd_joint6" type="revolute">
   <origin xyz="0.118077 0.110626 0.04364" rpy="0 0 0"/>
   <parent link="hd_link5"/>
   <child link="hd_link6"/>
   <axis xyz="0.115545 0.98806 -0.101919"/>
+  <xacro:insert_block name="joint6_limits"/>
 </joint>
 <joint name="hd_joint7" type="fixed">
