Commit message: new urdf with correct link lengths

File: kinematics/new_description/urdf/onyx.urdf.xacro (robot description, xacro)
@@ -1,7 +1,8 @@
 <?xml version="1.0" ?>
 <robot name="onyx" xmlns:xacro="http://www.ros.org/wiki/xacro">
-<xacro:include filename="$(find new_description)/urdf/materials.xacro" />
+<!-- <xacro:include filename="$(find new_description)/urdf/materials.xacro" /> -->
 <!-- <xacro:include filename="$(find new_description)/urdf/onyx.trans" /> -->
-<xacro:include filename="$(find new_description)/urdf/onyx.gazebo" />
+<!-- <xacro:include filename="$(find new_description)/urdf/onyx.gazebo" /> -->
+<xacro:include filename="$(find new_description)/urdf/body.urdf.xacro" />
 <xacro:property name="rpm_to_Radps" value="${2*pi/60.0}" />     <!-- rotations per minute to Rad per second conversion -->
 <xacro:property name="velocity_scaling" value="8" />     <!-- allows to scale all max velocities down at once -->
@@ -30,62 +31,21 @@
   <xacro:aaa_joint_limits lower="${-pi}" upper="${pi}" velocity="${10 * rpm_to_Radps}" />
 </xacro:property>
-<link name="base_link">
-  <inertial>
-    <origin xyz="0 0 0" rpy="0 0 0"/>
-    <mass value="10"/>
-    <!-- <inertia ixx="0.00171" iyy="0.00171" izz="0.003332" ixy="-0.0" iyz="0.0" ixz="0.0"/> -->
-    <inertia ixx="0.866667" iyy="0.241667" izz="11.4583" ixy="0" iyz="0" ixz="0"/>
-  </inertial>
-  <visual>
-    <origin xyz="0 0 0" rpy="0 0 0"/>
-    <geometry>
-      <box size="0.5 1 0.2"/>
-    </geometry>
-    <material name="silver"/>
-  </visual>
-  <collision>
-    <origin xyz="0 0 0" rpy="0 0 0"/>
-    <geometry>
-      <box size="0.5 1 0.2"/>
-    </geometry>
-  </collision>
-</link>
-<link name="link0">
-  <inertial>
-    <origin xyz="1.1956123958086707e-13 -3.565798973482466e-17 0.006224605561972922" rpy="0 0 0"/>
-    <mass value="1.001112718637754"/>
-    <inertia ixx="0.00171" iyy="0.00171" izz="0.003332" ixy="-0.0" iyz="0.0" ixz="0.0"/>
-  </inertial>
-  <visual>
-    <origin xyz="0 0 0" rpy="0 0 0"/>
-    <geometry>
-      <mesh filename="file://$(find new_description)/new_meshes/base_link.stl" scale="0.001 0.001 0.001"/>
-    </geometry>
-    <material name="silver"/>
-  </visual>
-  <collision>
-    <origin xyz="0 0 0" rpy="0 0 0"/>
-    <geometry>
-      <mesh filename="file://$(find new_description)/new_meshes/base_link.stl" scale="0.001 0.001 0.001"/>
-    </geometry>
-  </collision>
-</link>
 <link name="link1">
   <inertial>
-    <origin xyz="-0.021682763192533625 -0.00019343861423738655 -0.1015440461378264" rpy="0 0 0"/>
+    <origin xyz="0.00019343861423741504 0.02168276319253362 0.10154404613782692" rpy="0 0 0"/>
     <mass value="4.6341269008415775"/>
-    <inertia ixx="0.020818" iyy="0.028645" izz="0.018526" ixy="9.3e-05" iyz="8e-06" ixz="-0.002659"/>
-  </inertial>
-  <visual>
-    <origin xyz="-0.0 -0.0 -0.0" rpy="0 0 0"/>
-    <geometry>
-      <mesh filename="file://$(find new_description)/new_meshes/2j_simplified_v2_1.stl" scale="0.001 0.001 0.001"/>
-    </geometry>
-    <material name="silver"/>
-  </visual>
-  <collision>
-    <origin xyz="-0.0 -0.0 -0.0" rpy="0 0 0"/>
-    <geometry>
-      <mesh filename="file://$(find new_description)/new_meshes/2j_simplified_v2_1.stl" scale="0.001 0.001 0.001"/>
+    <inertia ixx="0.028645" iyy="0.020818" izz="0.018526" ixy="9.3e-05" iyz="-0.002659" ixz="8e-06"/>
+  </inertial>
+  <visual>
+    <origin xyz="0.07 0.2225 -0.195" rpy="0 0 0"/>
+    <geometry>
+      <mesh filename="file://$(find new_description)/meshes/1._J1J2_v2_v2_1.stl" scale="0.001 0.001 0.001"/>
+    </geometry>
+    <material name="silver"/>
+  </visual>
+  <collision>
+    <origin xyz="0.07 0.2225 -0.195" rpy="0 0 0"/>
+    <geometry>
+      <mesh filename="file://$(find new_description)/meshes/1._J1J2_v2_v2_1.stl" scale="0.001 0.001 0.001"/>
     </geometry>
   </collision>
@@ -93,19 +53,19 @@
 <link name="link2">
   <inertial>
-    <origin xyz="0.011067557585023063 -0.18599999999999753 -3.608224830031759e-16" rpy="0 0 0"/>
-    <mass value="3.1139206406559206"/>
-    <inertia ixx="0.069339" iyy="0.005977" izz="0.067529" ixy="-0.0" iyz="-0.0" ixz="-0.0"/>
-  </inertial>
-  <visual>
-    <origin xyz="0.1185 0.0 0.1185" rpy="0 0 0"/>
-    <geometry>
-      <mesh filename="file://$(find new_description)/new_meshes/1.2_tube_1_single_component_v2_1.stl" scale="0.001 0.001 0.001"/>
-    </geometry>
-    <material name="silver"/>
-  </visual>
-  <collision>
-    <origin xyz="0.1185 0.0 0.1185" rpy="0 0 0"/>
-    <geometry>
-      <mesh filename="file://$(find new_description)/new_meshes/1.2_tube_1_single_component_v2_1.stl" scale="0.001 0.001 0.001"/>
+    <origin xyz="-1.3322676295501878e-15 -0.011073644011486264 0.18649999999999678" rpy="0 0 0"/>
+    <mass value="3.117767835019512"/>
+    <inertia ixx="0.067945" iyy="0.069755" izz="0.005983" ixy="0.0" iyz="-0.0" ixz="0.0"/>
+  </inertial>
+  <visual>
+    <origin xyz="0.07 0.104 -0.3135" rpy="0 0 0"/>
+    <geometry>
+      <mesh filename="file://$(find new_description)/meshes/1.1_bras_1_single_c_v3_1.stl" scale="0.001 0.001 0.001"/>
+    </geometry>
+    <material name="silver"/>
+  </visual>
+  <collision>
+    <origin xyz="0.07 0.104 -0.3135" rpy="0 0 0"/>
+    <geometry>
+      <mesh filename="file://$(find new_description)/meshes/1.1_bras_1_single_c_v3_1.stl" scale="0.001 0.001 0.001"/>
     </geometry>
   </collision>
@@ -113,19 +73,19 @@
 <link name="link3">
   <inertial>
-    <origin xyz="0.10154404613781516 -0.021682763192532595 0.00019343861423570807" rpy="0 0 0"/>
+    <origin xyz="0.00019343861423579134 -0.101544046137815 0.021682763192532706" rpy="0 0 0"/>
     <mass value="4.6341269008415775"/>
-    <inertia ixx="0.018526" iyy="0.020818" izz="0.028645" ixy="0.002659" iyz="-9.3e-05" ixz="8e-06"/>
-  </inertial>
-  <visual>
-    <origin xyz="0.1185 0.372 0.1185" rpy="0 0 0"/>
-    <geometry>
-      <mesh filename="file://$(find new_description)/new_meshes/2j_simplified_v2_2.stl" scale="0.001 0.001 0.001"/>
-    </geometry>
-    <material name="silver"/>
-  </visual>
-  <collision>
-    <origin xyz="0.1185 0.372 0.1185" rpy="0 0 0"/>
-    <geometry>
-      <mesh filename="file://$(find new_description)/new_meshes/2j_simplified_v2_2.stl" scale="0.001 0.001 0.001"/>
+    <inertia ixx="0.028645" iyy="0.018526" izz="0.020818" ixy="-8e-06" iyz="0.002659" ixz="9.3e-05"/>
+  </inertial>
+  <visual>
+    <origin xyz="0.07 0.104 -0.6865" rpy="0 0 0"/>
+    <geometry>
+      <mesh filename="file://$(find new_description)/meshes/1._J1J2_v2_v2_2.stl" scale="0.001 0.001 0.001"/>
+    </geometry>
+    <material name="silver"/>
+  </visual>
+  <collision>
+    <origin xyz="0.07 0.104 -0.6865" rpy="0 0 0"/>
+    <geometry>
+      <mesh filename="file://$(find new_description)/meshes/1._J1J2_v2_v2_2.stl" scale="0.001 0.001 0.001"/>
     </geometry>
   </collision>
@@ -133,19 +93,19 @@
 <link name="link4">
   <inertial>
-    <origin xyz="0.003331504937314443 -0.15487679697152384 4.925226892993351e-14" rpy="0 0 0"/>
-    <mass value="2.3051495546208427"/>
-    <inertia ixx="0.027883" iyy="0.004302" izz="0.026991" ixy="0.00098" iyz="0.0" ixz="-0.0"/>
-  </inertial>
-  <visual>
-    <origin xyz="0.0 0.4905 0.1185" rpy="0 0 0"/>
-    <geometry>
-      <mesh filename="file://$(find new_description)/new_meshes/1.2_tube_2_single_component_v2_1.stl" scale="0.001 0.001 0.001"/>
-    </geometry>
-    <material name="silver"/>
-  </visual>
-  <collision>
-    <origin xyz="0.0 0.4905 0.1185" rpy="0 0 0"/>
-    <geometry>
-      <mesh filename="file://$(find new_description)/new_meshes/1.2_tube_2_single_component_v2_1.stl" scale="0.001 0.001 0.001"/>
+    <origin xyz="4.5352610555937645e-14 -0.0030701810090929815 0.18321907839266705" rpy="0 0 0"/>
+    <mass value="2.501356467163731"/>
+    <inertia ixx="0.0397" iyy="0.040591" izz="0.004603" ixy="0.0" iyz="0.001154" ixz="-0.0"/>
+  </inertial>
+  <visual>
+    <origin xyz="0.07 0.2225 -0.805" rpy="0 0 0"/>
+    <geometry>
+      <mesh filename="file://$(find new_description)/meshes/1._tube_2_single_component_v2_1.stl" scale="0.001 0.001 0.001"/>
+    </geometry>
+    <material name="silver"/>
+  </visual>
+  <collision>
+    <origin xyz="0.07 0.2225 -0.805" rpy="0 0 0"/>
+    <geometry>
+      <mesh filename="file://$(find new_description)/meshes/1._tube_2_single_component_v2_1.stl" scale="0.001 0.001 0.001"/>
     </geometry>
   </collision>
@@ -153,19 +113,19 @@
 <link name="link5">
   <inertial>
-    <origin xyz="-0.10154404613785854 -0.021682763192527488 -0.00019343861423763709" rpy="0 0 0"/>
+    <origin xyz="-0.00019343861423758157 0.10154404613786167 0.021682763192527377" rpy="0 0 0"/>
     <mass value="4.6341269008415775"/>
-    <inertia ixx="0.018526" iyy="0.020818" izz="0.028645" ixy="-0.002659" iyz="9.3e-05" ixz="8e-06"/>
-  </inertial>
-  <visual>
-    <origin xyz="-0.016 0.7625 0.1185" rpy="0 0 0"/>
-    <geometry>
-      <mesh filename="file://$(find new_description)/new_meshes/2j_simplified_v2_3.stl" scale="0.001 0.001 0.001"/>
-    </geometry>
-    <material name="silver"/>
-  </visual>
-  <collision>
-    <origin xyz="-0.016 0.7625 0.1185" rpy="0 0 0"/>
-    <geometry>
-      <mesh filename="file://$(find new_description)/new_meshes/2j_simplified_v2_3.stl" scale="0.001 0.001 0.001"/>
+    <inertia ixx="0.028645" iyy="0.018526" izz="0.020818" ixy="-8e-06" iyz="-0.002659" ixz="-9.3e-05"/>
+  </inertial>
+  <visual>
+    <origin xyz="0.07 0.2385 -1.128" rpy="0 0 0"/>
+    <geometry>
+      <mesh filename="file://$(find new_description)/meshes/1._J1J2_v2_v2_3.stl" scale="0.001 0.001 0.001"/>
+    </geometry>
+    <material name="silver"/>
+  </visual>
+  <collision>
+    <origin xyz="0.07 0.2385 -1.128" rpy="0 0 0"/>
+    <geometry>
+      <mesh filename="file://$(find new_description)/meshes/1._J1J2_v2_v2_3.stl" scale="0.001 0.001 0.001"/>
     </geometry>
   </collision>
@@ -173,19 +133,39 @@
 <link name="link6">
   <inertial>
-    <origin xyz="-0.0003178609482610145 -0.06769985638413722 -0.0002575140808085824" rpy="0 0 0"/>
+    <origin xyz="-0.0003178609482202416 -0.000257514080764229 0.06769985638413734" rpy="0 0 0"/>
     <mass value="0.236737000660016"/>
-    <inertia ixx="0.000328" iyy="0.00022" izz="0.000476" ixy="4e-06" iyz="-1e-06" ixz="0.0"/>
-  </inertial>
-  <visual>
-    <origin xyz="0.1025 0.881 0.1185" rpy="0 0 0"/>
-    <geometry>
-      <mesh filename="file://$(find new_description)/new_meshes/1.2_gripper_single_component_v2_1.stl" scale="0.001 0.001 0.001"/>
-    </geometry>
-    <material name="silver"/>
-  </visual>
-  <collision>
-    <origin xyz="0.1025 0.881 0.1185" rpy="0 0 0"/>
-    <geometry>
-      <mesh filename="file://$(find new_description)/new_meshes/1.2_gripper_single_component_v2_1.stl" scale="0.001 0.001 0.001"/>
+    <inertia ixx="0.000328" iyy="0.000476" izz="0.00022" ixy="0.0" iyz="1e-06" ixz="-4e-06"/>
+  </inertial>
+  <visual>
+    <origin xyz="0.07 0.12 -1.2465" rpy="0 0 0"/>
+    <geometry>
+      <mesh filename="file://$(find new_description)/meshes/Gripper_no_torque_sensor_v2_1.stl" scale="0.001 0.001 0.001"/>
+    </geometry>
+    <material name="silver"/>
+  </visual>
+  <collision>
+    <origin xyz="0.07 0.12 -1.2465" rpy="0 0 0"/>
+    <geometry>
+      <mesh filename="file://$(find new_description)/meshes/Gripper_no_torque_sensor_v2_1.stl" scale="0.001 0.001 0.001"/>
+    </geometry>
+  </collision>
+</link>
+<link name="Arm_A_v6_2">
+  <inertial>
+    <origin xyz="0.01895133656783434 0.003750000076247456 0.034431297042308184" rpy="0 0 0"/>
+    <mass value="0.11091056155247334"/>
+    <inertia ixx="0.000106" iyy="0.000118" izz="1.4e-05" ixy="-0.0" iyz="-0.0" ixz="1.1e-05"/>
+  </inertial>
+  <visual>
+    <origin xyz="0.055 0.0975 -1.328" rpy="0 0 0"/>
+    <geometry>
+      <mesh filename="file://$(find new_description)/meshes/Arm_A_v6_2.stl" scale="0.001 0.001 0.001"/>
+    </geometry>
+    <material name="silver"/>
+  </visual>
+  <collision>
+    <origin xyz="0.055 0.0975 -1.328" rpy="0 0 0"/>
+    <geometry>
+      <mesh filename="file://$(find new_description)/meshes/Arm_A_v6_2.stl" scale="0.001 0.001 0.001"/>
     </geometry>
   </collision>
@@ -193,156 +173,130 @@
 <link name="Arm_A_v6_1">
   <inertial>
-    <origin xyz="0.01895133656779084 -0.03443129704231196 -0.003749999923799513" rpy="0 0 0"/>
+    <origin xyz="-0.018951336567834404 0.0037499999238455595 0.034431297042308406" rpy="0 0 0"/>
     <mass value="0.11091056155247334"/>
-    <inertia ixx="0.000106" iyy="1.4e-05" izz="0.000118" ixy="-1.1e-05" iyz="0.0" ixz="-0.0"/>
-  </inertial>
-  <visual>
-    <origin xyz="0.0875 0.9625 0.141" rpy="0 0 0"/>
-    <geometry>
-      <mesh filename="file://$(find new_description)/new_meshes/Arm_A_v6_1.stl" scale="0.001 0.001 0.001"/>
-    </geometry>
-    <material name="silver"/>
-  </visual>
-  <collision>
-    <origin xyz="0.0875 0.9625 0.141" rpy="0 0 0"/>
-    <geometry>
-      <mesh filename="file://$(find new_description)/new_meshes/Arm_A_v6_1.stl" scale="0.001 0.001 0.001"/>
-    </geometry>
-  </collision>
-</link>
-<link name="Arm_A_v6_2">
-  <inertial>
-    <origin xyz="-0.018951336567878035 -0.03443129704230807 -0.0037500000762014374" rpy="0 0 0"/>
-    <mass value="0.11091056155247334"/>
-    <inertia ixx="0.000106" iyy="1.4e-05" izz="0.000118" ixy="1.1e-05" iyz="-0.0" ixz="-0.0"/>
-  </inertial>
-  <visual>
-    <origin xyz="0.1175 0.9625 0.141" rpy="0 0 0"/>
-    <geometry>
-      <mesh filename="file://$(find new_description)/new_meshes/Arm_A_v6_2.stl" scale="0.001 0.001 0.001"/>
-    </geometry>
-    <material name="silver"/>
-  </visual>
-  <collision>
-    <origin xyz="0.1175 0.9625 0.141" rpy="0 0 0"/>
-    <geometry>
-      <mesh filename="file://$(find new_description)/new_meshes/Arm_A_v6_2.stl" scale="0.001 0.001 0.001"/>
-    </geometry>
-  </collision>
-</link>
-<link name="Hand_v3_2">
-  <inertial>
-    <origin xyz="0.00933673220576138 -8.5407306888996e-06 0.022500003616503783" rpy="0 0 0"/>
+    <inertia ixx="0.000106" iyy="0.000118" izz="1.4e-05" ixy="-0.0" iyz="0.0" ixz="-1.1e-05"/>
+  </inertial>
+  <visual>
+    <origin xyz="0.085 0.0975 -1.328" rpy="0 0 0"/>
+    <geometry>
+      <mesh filename="file://$(find new_description)/meshes/Arm_A_v6_1.stl" scale="0.001 0.001 0.001"/>
+    </geometry>
+    <material name="silver"/>
+  </visual>
+  <collision>
+    <origin xyz="0.085 0.0975 -1.328" rpy="0 0 0"/>
+    <geometry>
+      <mesh filename="file://$(find new_description)/meshes/Arm_A_v6_1.stl" scale="0.001 0.001 0.001"/>
+    </geometry>
+  </collision>
+</link>
+<link name="Finger_v1_2">
+  <inertial>
+    <origin xyz="0.009336732205807656 -0.02249999638344631 8.540730686679154e-06" rpy="0 0 0"/>
     <mass value="0.21086382762249625"/>
-    <inertia ixx="3.4e-05" iyy="5.6e-05" izz="3.6e-05" ixy="-0.0" iyz="-0.0" ixz="0.0"/>
-  </inertial>
-  <visual>
-    <origin xyz="0.084582 1.04908 0.141" rpy="0 0 0"/>
-    <geometry>
-      <mesh filename="file://$(find new_description)/new_meshes/Finger_v1_1.stl" scale="0.001 0.001 0.001"/>
-    </geometry>
-    <material name="silver"/>
-  </visual>
-  <collision>
-    <origin xyz="0.084582 1.04908 0.141" rpy="0 0 0"/>
-    <geometry>
-      <mesh filename="file://$(find new_description)/new_meshes/Finger_v1_1.stl" scale="0.001 0.001 0.001"/>
-    </geometry>
-  </collision>
-</link>
-<link name="Hand_v3_1">
-  <inertial>
-    <origin xyz="-0.009336732205854098 -8.540730685568931e-06 0.02249999638349527" rpy="0 0 0"/>
+    <inertia ixx="3.4e-05" iyy="3.6e-05" izz="5.6e-05" ixy="0.0" iyz="0.0" ixz="0.0"/>
+  </inertial>
+  <visual>
+    <origin xyz="0.052082 0.0975 -1.41458" rpy="0 0 0"/>
+    <geometry>
+      <mesh filename="file://$(find new_description)/meshes/Finger_v1_2.stl" scale="0.001 0.001 0.001"/>
+    </geometry>
+    <material name="silver"/>
+  </visual>
+  <collision>
+    <origin xyz="0.052082 0.0975 -1.41458" rpy="0 0 0"/>
+    <geometry>
+      <mesh filename="file://$(find new_description)/meshes/Finger_v1_2.stl" scale="0.001 0.001 0.001"/>
+    </geometry>
+  </collision>
+</link>
+<link name="Finger_v1_1">
+  <inertial>
+    <origin xyz="-0.009336732205807885 -0.02250000361645496 8.540730686901199e-06" rpy="0 0 0"/>
     <mass value="0.21086382762249625"/>
-    <inertia ixx="3.4e-05" iyy="5.6e-05" izz="3.6e-05" ixy="0.0" iyz="0.0" ixz="0.0"/>
-  </inertial>
-  <visual>
-    <origin xyz="0.120418 1.04908 0.141" rpy="0 0 0"/>
-    <geometry>
-      <mesh filename="file://$(find new_description)/new_meshes/Finger_v1_2.stl" scale="0.001 0.001 0.001"/>
-    </geometry>
-    <material name="silver"/>
-  </visual>
-  <collision>
-    <origin xyz="0.120418 1.04908 0.141" rpy="0 0 0"/>
-    <geometry>
-      <mesh filename="file://$(find new_description)/new_meshes/Finger_v1_2.stl" scale="0.001 0.001 0.001"/>
-    </geometry>
-  </collision>
-</link>
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