Commit message: normal limits in urdf

File: kinematics/new_description/urdf/onyx.urdf.xacro (robot description, xacro)
@@ -5,25 +5,25 @@
 <xacro:include filename="$(find new_description)/urdf/onyx.gazebo" />
 <xacro:property name="rpm_to_Radps" value="${2*pi/60.0}" />     <!-- rotations per minute to Rad per second conversion -->
-<xacro:property name="velocity_scaling" value="0.8" />     <!-- allows to scale all max velocities down at once -->
+<xacro:property name="velocity_scaling" value="8" />     <!-- allows to scale all max velocities down at once -->
 <xacro:macro name="aaa_joint_limits" params="lower:=0.0 upper:=0.0 velocity:=${rpm_to_Radps} effort:=100.0">
   <limit lower="${lower}" upper="${upper}" velocity="${velocity}" effort="${effort}"/>
 </xacro:macro>
 <xacro:property name="joint1_limits">
-  <xacro:aaa_joint_limits lower="${-4/7*pi}" upper="${0}" velocity="${1.83 * rpm_to_Radps * velocity_scaling}" />
+  <xacro:aaa_joint_limits lower="${-3/2*pi}" upper="${3/2*pi}" velocity="${1.83 * rpm_to_Radps * velocity_scaling}" />
 </xacro:property>
 <xacro:property name="joint2_limits">
-  <xacro:aaa_joint_limits lower="${-1.92}" upper="${0}" velocity="${1.377 * rpm_to_Radps * velocity_scaling}" />
+  <xacro:aaa_joint_limits lower="${-pi}" upper="${pi}" velocity="${1.377 * rpm_to_Radps * velocity_scaling}" />
 </xacro:property>
 <xacro:property name="joint3_limits">
-  <xacro:aaa_joint_limits lower="${-pi}" upper="${0}" velocity="${1.377 * rpm_to_Radps * velocity_scaling}" />
+  <xacro:aaa_joint_limits lower="${-pi}" upper="${pi}" velocity="${1.377 * rpm_to_Radps * velocity_scaling}" />
 </xacro:property>
 <xacro:property name="joint4_limits">
-  <xacro:aaa_joint_limits lower="${-pi}" upper="${1/2*pi}" velocity="${1.83 * rpm_to_Radps * velocity_scaling}" />
+  <xacro:aaa_joint_limits lower="${-3/2*pi}" upper="${3/2*pi}" velocity="${1.83 * rpm_to_Radps * velocity_scaling}" />
 </xacro:property>
 <xacro:property name="joint5_limits">
-  <xacro:aaa_joint_limits lower="${-1.92}" upper="${0}" velocity="${1.83 * rpm_to_Radps * velocity_scaling}" />
+  <xacro:aaa_joint_limits lower="${-pi}" upper="${pi}" velocity="${1.83 * rpm_to_Radps * velocity_scaling}" />
 </xacro:property>
 <xacro:property name="joint6_limits">
-  <xacro:aaa_joint_limits lower="${-pi}" upper="${pi}" velocity="${1.83 * rpm_to_Radps * velocity_scaling}" />
+  <xacro:aaa_joint_limits lower="${-3/2*pi}" upper="${3/2*pi}" velocity="${1.83 * rpm_to_Radps * velocity_scaling}" />
 </xacro:property>
 <xacro:property name="finger_limits">

Commit message: j1 limit in urdf

File: kinematics/new_description/urdf/onyx.urdf.xacro (robot description, xacro)
@@ -6,10 +6,10 @@
 <xacro:include filename="$(find new_description)/urdf/body.urdf.xacro" />
 <xacro:property name="rpm_to_Radps" value="${2*pi/60.0}" />     <!-- rotations per minute to Rad per second conversion -->
-<xacro:property name="velocity_scaling" value="8" />     <!-- allows to scale all max velocities down at once -->
+<xacro:property name="velocity_scaling" value="0.8" />     <!-- allows to scale all max velocities down at once -->
 <xacro:macro name="aaa_joint_limits" params="lower:=0.0 upper:=0.0 velocity:=${rpm_to_Radps} effort:=100.0">
   <limit lower="${lower}" upper="${upper}" velocity="${velocity}" effort="${effort}"/>
 </xacro:macro>
 <xacro:property name="joint1_limits">
-  <xacro:aaa_joint_limits lower="${-3/2*pi}" upper="${3/2*pi}" velocity="${1.83 * rpm_to_Radps * velocity_scaling}" />
+  <xacro:aaa_joint_limits lower="${-pi/2}" upper="${pi/2}" velocity="${1.83 * rpm_to_Radps * velocity_scaling}" />
 </xacro:property>
 <xacro:property name="joint2_limits">

Commit message: avoid collision and trying gazebo hardware interface

File: kinematics/new_description/urdf/onyx.urdf.xacro (robot description, xacro)
@@ -5,5 +5,6 @@
 <!-- <xacro:include filename="$(find new_description)/urdf/onyx.gazebo" /> -->
 <xacro:include filename="$(find new_description)/urdf/body.urdf.xacro" />
-<xacro:property name="rpm_to_Radps" value="${2*pi/60.0}" />     <!-- rotations per minute to Rad per second conversion -->
+<xacro:include filename="$(find rover_description)/description/kerby.gazebo" />
+<xacro:property name="rpm_to_Radps" value="${2*pi/60.0}"/>     <!-- rotations per minute to Rad per second conversion  -->
 <xacro:property name="velocity_scaling" value="1.0" />     <!-- allows to scale all max velocities down at once -->
 <xacro:macro name="aaa_joint_limits" params="lower:=0.0 upper:=0.0 velocity:=${rpm_to_Radps} effort:=100.0">

File: kinematics/new_moveit_config/config/kerby.ros2_control.xacro (robot description, xacro)
@@ -6,5 +6,6 @@
             <hardware>
                 <!-- By default, set up controllers for simulation. This won't work on real hardware -->
-                <plugin>kerby_hw_interface/KerbyArmInterface</plugin>
+                <plugin>gazebo_ros2_control/GazeboSystem</plugin>
+                <!-- <plugin>kerby_hw_interface/KerbyArmInterface</plugin> -->
             </hardware>
             <joint name="hd_joint1">
@@ -50,17 +51,10 @@
                 <state_interface name="velocity"/>
             </joint>
-            <joint name="finger_joint1">
-                <command_interface name="position"/>
-                <state_interface name="position">
-                  <param name="initial_value">${initial_positions['finger_joint1']}</param>
-                </state_interface>
-                <state_interface name="velocity"/>
-            </joint>
         </ros2_control>
-        <!-- <gazebo>
+        <gazebo>
           <plugin name="gazebo_ros2_control" filename="libgazebo_ros2_control.so">
-              <parameters>$(find new_descriptioni)/config/ros2_controllers.yaml</parameters>
+              <parameters>$(find new_moveit_config)/config/ros2_controllers.yaml</parameters>
           </plugin>
-        </gazebo>   -->
+        </gazebo>
         <gazebo>
           <plugin name="rover_joint_state" filename="libgazebo_ros_joint_state_publisher.so">

Commit message: small modif urdf xacro

File: kinematics/new_description/urdf/onyx.urdf.xacro (robot description, xacro)
@@ -7,27 +7,27 @@
 <xacro:property name="rpm_to_Radps" value="${2*pi/60.0}" />     <!-- rotations per minute to Rad per second conversion -->
 <xacro:property name="velocity_scaling" value="1.0" />     <!-- allows to scale all max velocities down at once -->
-<xacro:macro name="aaa_joint_limits" params="lower:=0.0 upper:=0.0 velocity:=${rpm_to_Radps} effort:=100.0">
+<xacro:macro name="joint_limits" params="lower:=0.0 upper:=0.0 velocity:=${rpm_to_Radps} effort:=100.0">
   <limit lower="${lower}" upper="${upper}" velocity="${velocity}" effort="${effort}"/>
 </xacro:macro>
 <xacro:property name="joint1_limits">
-  <xacro:aaa_joint_limits lower="${-pi}" upper="${pi}" velocity="${1.83 * rpm_to_Radps * velocity_scaling}" />
+  <xacro:joint_limits lower="${-pi}" upper="${pi}" velocity="${1.83 * rpm_to_Radps * velocity_scaling}" />
 </xacro:property>
 <xacro:property name="joint2_limits">
-  <xacro:aaa_joint_limits lower="${-pi}" upper="${pi}" velocity="${1.377 * rpm_to_Radps * velocity_scaling}" />
+  <xacro:joint_limits lower="${-pi}" upper="${pi}" velocity="${1.377 * rpm_to_Radps * velocity_scaling}" />
 </xacro:property>
 <xacro:property name="joint3_limits">
-  <xacro:aaa_joint_limits lower="${-pi}" upper="${pi}" velocity="${1.377 * rpm_to_Radps * velocity_scaling}" />
+  <xacro:joint_limits lower="${-pi}" upper="${pi}" velocity="${1.377 * rpm_to_Radps * velocity_scaling}" />
 </xacro:property>
 <xacro:property name="joint4_limits">
-  <xacro:aaa_joint_limits lower="${-3/2*pi}" upper="${3/2*pi}" velocity="${1.83 * rpm_to_Radps * velocity_scaling}" />
+  <xacro:joint_limits lower="${-3/2*pi}" upper="${3/2*pi}" velocity="${1.83 * rpm_to_Radps * velocity_scaling}" />
 </xacro:property>
 <xacro:property name="joint5_limits">
-  <xacro:aaa_joint_limits lower="${-pi}" upper="${pi}" velocity="${1.83 * rpm_to_Radps * velocity_scaling}" />
+  <xacro:joint_limits lower="${-pi}" upper="${pi}" velocity="${1.83 * rpm_to_Radps * velocity_scaling}" />
 </xacro:property>
 <xacro:property name="joint6_limits">
-  <xacro:aaa_joint_limits lower="${-3/2*pi}" upper="${3/2*pi}" velocity="${1.83 * rpm_to_Radps * velocity_scaling}" />
+  <xacro:joint_limits lower="${-3/2*pi}" upper="${3/2*pi}" velocity="${1.83 * rpm_to_Radps * velocity_scaling}" />
 </xacro:property>
 <xacro:property name="finger_limits">
-  <xacro:aaa_joint_limits lower="${-pi}" upper="${pi}" velocity="${10 * rpm_to_Radps}" />
+  <xacro:joint_limits lower="${-pi}" upper="${pi}" velocity="${10 * rpm_to_Radps}" />
 </xacro:property>
 <link name="link1">
